Commit message: Added LIDAR

File: description/urdf/base.urdf.xacro (robot description, xacro)
@@ -59,22 +59,22 @@
     mass_kg="0.01"
   />
-  <!--     <link name="scan" />
-    <joint name="base_to_scan" type="fixed">
-      <parent link="base_link" />
-      <child link="scan" />
-      <origin xyz="-0.018  -0.090 0.430" rpy="0 0 ${M_PI}" />
-    </joint>
-    <xacro:ld06 lidar_prefix="top_lidar">
-        <origin xyz="0 0 0" rpy="0 0 0" />
-    </xacro:ld06>
-    <joint name="base_to_lidar_frame_top_lidar" type="fixed">
-      <parent link="scan" />
-      <child link="lidar_frame_top_lidar" />
-      <origin xyz="0 0 0" rpy="0 0 0" />
-    </joint>
-    <xacro:diff_drive_controller
-        wheel_separation="${wheel_pos_y * 2}"
-        wheel_radius="${wheel_radius}"
-    /> -->
+  <link name="scan" />
+  <joint name="base_to_scan" type="fixed">
+    <parent link="base_link" />
+    <child link="scan" />
+    <origin xyz="0.155 0 0.305" rpy="0 0 ${M_PI}" />
+  </joint>
+  <xacro:ld06 lidar_prefix="top_lidar">
+    <origin xyz="0 0 0" rpy="0 0 0" />
+  </xacro:ld06>
+  <joint name="base_to_lidar_frame_top_lidar" type="fixed">
+    <parent link="scan" />
+    <child link="lidar_frame_top_lidar" />
+    <origin xyz="0 0 0" rpy="0 0 0" />
+  </joint>
+  <xacro:diff_drive_controller
+    wheel_separation="${wheel_pos_y * 2}"
+    wheel_radius="${wheel_radius}"
+  />
   <!--
 Copyright (c) 2024 Michael Wimble

Commit message: Fixed LIDAR in URDF

File: description/urdf/base.urdf.xacro (robot description, xacro)
@@ -63,5 +63,5 @@
     <parent link="base_link" />
     <child link="scan" />
-    <origin xyz="0.155 0 0.305" rpy="0 0 ${M_PI}" />
+    <origin xyz="0.155 0 0.305" rpy="0 0 -${M_PI / 2}" />
   </joint>
   <xacro:ld06 lidar_prefix="top_lidar">
@@ -71,5 +71,5 @@
     <parent link="scan" />
     <child link="lidar_frame_top_lidar" />
-    <origin xyz="0 0 0" rpy="0 0 0" />
+    <origin xyz="0 0 0" rpy="0 0 -${M_PI / 2}" />
   </joint>
   <xacro:diff_drive_controller

Commit message: Basic simulation started

File: description/urdf/base.urdf.xacro (robot description, xacro)
@@ -10,4 +10,12 @@
   <xacro:include filename="$(find description)/urdf/wheel.urdf.xacro" />
   <xacro:include filename="$(find description)/urdf/oakd.urdf.xacro" />
+  <xacro:arg name="use_ros2_control" default="true" />
+  <xacro:arg name="sim_mode" default="false" />
+  <xacro:if value="$(arg use_ros2_control)">
+    <xacro:include filename="ros2_control.xacro" />
+  </xacro:if>
+  <xacro:unless value="$(arg use_ros2_control)">
+    <xacro:include filename="gazebo_control.xacro" />
+  </xacro:unless>
   <link name="base_link">
     <collision>
@@ -24,5 +32,5 @@
       <origin rpy="0 0 0" xyz="0 0 ${(body_height/2)}" />
     </visual>
-    <xacro:solid_cylinder_inertial rpy="0 0 0" xyz="0 0 0.05" mass_kg="${mass}"
+    <xacro:solid_cylinder_inertial rpy="0 0 0" xyz="-0.05 0 0.05" mass_kg="${mass}"
       radius="${body_radius}" length="${body_height}" />
   </link>
@@ -57,5 +65,5 @@
   />
   <xacro:caster_wheel
-    mass_kg="0.01"
+    mass_kg="0.4"
   />
   <link name="scan" />

File: description/urdf/gazebo.urdf.xacro (robot description, xacro)
@@ -2,19 +2,27 @@
   <xacro:macro name="diff_drive_controller" params="wheel_separation wheel_radius">
     <gazebo>
-      <plugin name="differential_drive_controller" filename="libgazebo_ros_diff_drive.so">
-        <ros>
-          <argument>odom:=odom/unfiltered</argument>
-        </ros>
-        <updateRate>100</updateRate>
+      <plugin name="gz::sim::systems::DiffDrive" filename="gz-sim-diff-drive-system">
+        <!-- Wheel Information -->
         <left_joint>left_wheel_joint</left_joint>
         <right_joint>right_wheel_joint</right_joint>
         <wheel_separation>${wheel_separation}</wheel_separation>
-        <wheel_diameter>${wheel_radius * 2}</wheel_diameter>
-        <max_wheel_acceleration>1.0</max_wheel_acceleration>
-        <robot_base_frame>base_footprint</robot_base_frame>
-        <publish_odom>true</publish_odom>
-        <publish_odom_tf>false</publish_odom_tf>
-        <publish_wheel_tf>true</publish_wheel_tf>
-        <odometry_frame>odom</odometry_frame>
+        <wheel_radius>${wheel_radius}</wheel_radius>
+        <!-- Limits -->
+        <!-- <max_wheel_torque>200</max_wheel_torque> -->
+        <max_linear_acceleration>1.0</max_linear_acceleration>
+        <!-- Input -->
+        <topic>cmd_vel</topic>
+        <!-- Output -->
+        <frame_id>odom</frame_id>
+        <child_frame_id>base_link</child_frame_id>
+        <odom_topic>odom</odom_topic>
+        <odom_publisher_frequency>30</odom_publisher_frequency>
+        <tf_topic>/tf</tf_topic>
+      </plugin>
+      <plugin filename="gz-sim-joint-state-publisher-system"
+        name="gz::sim::systems::JointStatePublisher">
+        <topic>joint_states</topic>
+        <joint_name>left_wheel_joint</joint_name>
+        <joint_name>right_wheel_joint</joint_name>
       </plugin>
     </gazebo>

File: description/urdf/ld06.urdf.xacro (robot description, xacro)
@@ -119,14 +119,13 @@
     </joint> -->
     <gazebo reference="lidar_frame_${lidar_prefix}">
+      <material>Gazebo/Black</material>
       <sensor name="sensor_ray_${lidar_prefix}" type="ray">
-        <always_on>true</always_on>
+        <pose> 0 0 0 0 0 0 </pose>
+        <visualize>true</visualize>
         <update_rate>10</update_rate>
-        <pose>0 0 0 0 0 0</pose>
-        <visualize>true</visualize>
-        <ray>
+        <lidar>
           <scan>
             <horizontal>
               <samples>450</samples>
-              <resolution>1.0</resolution>
               <min_angle>0</min_angle>
               <max_angle>6.28</max_angle>
@@ -136,29 +135,12 @@
             <min>0.05</min>
             <max>10.0</max>
-            <resolution>0.01</resolution>
           </range>
-          <!-- <noise>
-            <type>gaussian</type>
-            <mean>0.0</mean>
-            <stddev>0.02</stddev>
-          </noise> -->
-        </ray>
-        <plugin name="laserscan_${lidar_prefix}" filename="libgazebo_ros_ray_sensor.so">
-          <ros>
-            <remapping>~/out:=/scan_${lidar_prefix}</remapping>
-          </ros>
-          <always_on>true</always_on>
-          <frame_name>lidar_frame_${lidar_prefix}</frame_name>
-          <output_type>sensor_msgs/LaserScan</output_type>
-          <topic_name>/scan_${lidar_prefix}</topic_name>
-          <update_rate>10.0</update_rate>
-        </plugin>
+        </lidar>
+        <topic>/scan_${lidar_prefix}</topic>
+        <gz_frame_id>lidar_frame_${lidar_prefix}</gz_frame_id>
       </sensor>
-      <material>
-        Gazebo/Black
-      </material>
     </gazebo>
   </xacro:macro>
-<!--
+  <!--
 Copyright (c) 2024 Michael Wimble
 Permission is hereby granted, free of charge, to any person obtaining a copy

Commit message: Better sim with laser. Still not showing in gazebo.

File: description/urdf/base.urdf.xacro (robot description, xacro)
@@ -67,18 +67,14 @@
     mass_kg="0.4"
   />
-  <link name="scan" />
+  <!-- <link name="scan" />
   <joint name="base_to_scan" type="fixed">
     <parent link="base_link" />
     <child link="scan" />
     <origin xyz="0.155 0 0.305" rpy="0 0 -${M_PI / 2}" />
-  </joint>
+  </joint> -->
   <xacro:ld06 lidar_prefix="top_lidar">
-    <origin xyz="0 0 0" rpy="0 0 0" />
+    <!-- <origin xyz="0 0 0" rpy="0 0 0" /> -->
+    <origin xyz="0.155 0 0.305" rpy="0 0 -${M_PI / 2}" />
   </xacro:ld06>
-  <joint name="base_to_lidar_frame_top_lidar" type="fixed">
-    <parent link="scan" />
-    <child link="lidar_frame_top_lidar" />
-    <origin xyz="0 0 0" rpy="0 0 -${M_PI / 2}" />
-  </joint>
   <xacro:diff_drive_controller
     wheel_separation="${wheel_pos_y * 2}"

File: description/urdf/gazebo.urdf.xacro (robot description, xacro)
@@ -15,5 +15,5 @@
         <!-- Output -->
         <frame_id>odom</frame_id>
-        <child_frame_id>base_link</child_frame_id>
+        <child_frame_id>base_footprint</child_frame_id>
         <odom_topic>odom</odom_topic>
         <odom_publisher_frequency>30</odom_publisher_frequency>

File: description/urdf/ld06.urdf.xacro (robot description, xacro)
@@ -114,11 +114,16 @@
     </joint>
     <!-- <joint name="base_to_lidar_frame_${lidar_prefix}" type="fixed">
+      <parent link="scan" />
+      <child link="lidar_frame_${lidar_prefix}" />
+      <origin xyz="0 0 0" rpy="0 0 -${M_PI / 2}" />
+    </joint> -->
+    <joint name="base_to_lidar_frame_${lidar_prefix}" type="fixed">
       <parent link="base_link" />
       <child link="lidar_frame_${lidar_prefix}" />
       <xacro:insert_block name="joint_pose" />
-    </joint> -->
+    </joint>
     <gazebo reference="lidar_frame_${lidar_prefix}">
       <material>Gazebo/Black</material>
-      <sensor name="sensor_ray_${lidar_prefix}" type="gpu_lidar">
+      <sensor name="laser" type="gpu_lidar">
         <pose> 0 0 0 0 0 0 </pose>
         <visualize>true</visualize>
@@ -137,5 +142,5 @@
           </range>
         </lidar>
-        <topic>/scan_${lidar_prefix}</topic>
+        <topic>/scan</topic>
         <gz_frame_id>lidar_frame_${lidar_prefix}</gz_frame_id>
       </sensor>

Commit message: Basic sim lidar working again

File: description/urdf/base.urdf.xacro (robot description, xacro)
@@ -10,4 +10,5 @@
   <xacro:include filename="$(find description)/urdf/wheel.urdf.xacro" />
   <xacro:include filename="$(find description)/urdf/oakd.urdf.xacro" />
+  <xacro:include filename="$(find description)/urdf/lidar.xacro" />
   <xacro:arg name="use_ros2_control" default="true" />
   <xacro:arg name="sim_mode" default="false" />
@@ -18,5 +19,11 @@
     <xacro:include filename="gazebo_control.xacro" />
   </xacro:unless>
-  <link name="base_link">
+  <link name="base_link" />
+  <joint name="chassis_joint" type="fixed">
+    <origin xyz="0 0 0" rpy="0 0 0" />
+    <child link="chassis" />
+    <parent link="base_link" />
+  </joint>
+  <link name="chassis">
     <collision>
       <geometry>
@@ -35,5 +42,5 @@
       radius="${body_radius}" length="${body_height}" />
   </link>
-  <gazebo reference="base_link">
+  <gazebo reference="chassis">
     <material>
       Gazebo/Grey
@@ -43,6 +50,6 @@
   <joint name="base_footprint_joint" type="fixed">
     <origin xyz="0 0 ${base_to_floor_z_offset}" rpy="0 0 0" />
-    <parent link="base_footprint" />
-    <child link="base_link" />
+    <child link="base_footprint" />
+    <parent link="base_link" />
   </joint>
   <xacro:wheel
@@ -67,14 +74,7 @@
     mass_kg="0.4"
   />
-  <!-- <link name="scan" />
-  <joint name="base_to_scan" type="fixed">
-    <parent link="base_link" />
-    <child link="scan" />
+  <!-- <xacro:ld06 lidar_prefix="top_lidar">
     <origin xyz="0.155 0 0.305" rpy="0 0 -${M_PI / 2}" />
-  </joint> -->
-  <xacro:ld06 lidar_prefix="top_lidar">
-    <!-- <origin xyz="0 0 0" rpy="0 0 0" /> -->
-    <origin xyz="0.155 0 0.305" rpy="0 0 -${M_PI / 2}" />
-  </xacro:ld06>
+  </xacro:ld06> -->
   <xacro:diff_drive_controller
     wheel_separation="${wheel_pos_y * 2}"

File: description/urdf/caster.urdf.xacro (robot description, xacro)
@@ -31,5 +31,5 @@
     </gazebo>
     <joint name="caster_wheel_joint" type="fixed">
-      <parent link="base_link" />
+      <parent link="chassis" />
       <child link="caster_wheel_link" />
       <origin

File: description/urdf/gazebo.urdf.xacro (robot description, xacro)
@@ -15,5 +15,5 @@
         <!-- Output -->
         <frame_id>odom</frame_id>
-        <child_frame_id>base_footprint</child_frame_id>
+        <child_frame_id>base_link</child_frame_id>
         <odom_topic>odom</odom_topic>
         <odom_publisher_frequency>30</odom_publisher_frequency>

File: description/urdf/ros2_control.xacro (robot description, xacro)
@@ -1,5 +1,5 @@
 <?xml version="1.0"?>
 <robot xmlns:xacro="http://www.ros.org/wiki/xacro">
-  <xacro:unless value="$(arg sim_mode)">
+  <!-- <xacro:unless value="$(arg sim_mode)">
     <ros2_control name="RealRobot" type="system">
       <hardware>
@@ -30,6 +30,6 @@
       </joint>
     </ros2_control>
-  </xacro:unless>
-  <xacro:if value="$(arg sim_mode)">
+  </xacro:unless> -->
+  <!-- <xacro:if value="$(arg sim_mode)"> -->
     <ros2_control name="GazeboSystem" type="system">
       <hardware>
@@ -53,5 +53,5 @@
       </joint>
     </ros2_control>
-  </xacro:if>
+  <!-- </xacro:if> -->
   <gazebo>
     <plugin name="gz_ros2_control::GazeboSimROS2ControlPlugin"

Commit message: Changes for LIDAR in URDF

File: description/urdf/base.urdf.xacro (robot description, xacro)
@@ -10,5 +10,4 @@
   <xacro:include filename="$(find description)/urdf/wheel.urdf.xacro" />
   <xacro:include filename="$(find description)/urdf/oakd.urdf.xacro" />
-  <xacro:include filename="$(find description)/urdf/lidar.xacro" />
   <xacro:arg name="use_ros2_control" default="true" />
   <xacro:arg name="sim_mode" default="false" />
@@ -74,7 +73,7 @@
     mass_kg="0.4"
   />
-  <!-- <xacro:ld06 lidar_prefix="top_lidar">
-    <origin xyz="0.155 0 0.305" rpy="0 0 -${M_PI / 2}" />
-  </xacro:ld06> -->
+  <xacro:ld06 lidar_prefix="top_lidar">
+    <origin xyz="0.155 0 0.300" rpy="0 0 -${M_PI / 2}" />
+  </xacro:ld06>
   <xacro:diff_drive_controller
     wheel_separation="${wheel_pos_y * 2}"

File: description/urdf/ld06.urdf.xacro (robot description, xacro)
@@ -11,50 +11,15 @@
       <color rgba="0.05 0.05 0.2 1" />
     </material>
-    <xacro:property name="ldlidar_z_offset" value="-0.003" />
-    <xacro:property name="ld06_base_box_height" value="0.020" />
+    <xacro:property name="ld06_base_box_height" value="0.011" />
     <xacro:property name="ld06_base_box_width" value="0.060" />
     <xacro:property name="ld06_box_width" value="0.037" />
-    <xacro:property name="ld06_box_height" value="0.022" />
-    <xacro:property name="ld06_cylinder_height" value="0.013" />
+    <xacro:property name="ld06_box_height" value="0.020" />
+    <xacro:property name="ld06_cylinder_height" value="0.012" />
     <xacro:property name="ld06_cylinder_radius" value="0.015" />
-    <link name="ld06_box_${lidar_prefix}">
-      <collision>
-        <geometry>
-          <box size="${ld06_box_width} ${ld06_box_width} ${ld06_box_height}" />
-        </geometry>
-        <origin rpy="0 0 0" xyz="0 0 0" />
-      </collision>
-      <visual>
-        <geometry>
-          <box size="${ld06_box_width} ${ld06_box_width} ${ld06_box_height}" />
-        </geometry>
-        <origin rpy="0 0 0" xyz="0 0 0" />
-        <material name="ld06_${lidar_prefix}_blackish" />
-      </visual>
-    </link>
-    <gazebo reference="ld06_box_${lidar_prefix}">
-      <material>
-        Gazebo/Black
-      </material>
-    </gazebo>
-    <link name="ld06_cylinder_${lidar_prefix}">
-      <collision>
-        <geometry>
-          <cylinder radius="${ld06_cylinder_radius}" length="${ld06_cylinder_height}" />
-        </geometry>
-      </collision>
-      <visual>
-        <geometry>
-          <cylinder radius="${ld06_cylinder_radius}" length="${ld06_cylinder_height}" />
-        </geometry>
-        <origin xyz="0 0 0" rpy="0 0 0" />
-        <material name="ld06_${lidar_prefix}_cylinder" />
-      </visual>
-    </link>
-    <gazebo reference="ld06_cylinder_${lidar_prefix}">
-      <material>
-        Gazebo/BlueGlow
-      </material>
-    </gazebo>
+    <joint name="base_to_lidar_frame_${lidar_prefix}" type="fixed">
+      <parent link="base_link" />
+      <child link="lidar_frame_${lidar_prefix}" />
+      <xacro:insert_block name="joint_pose" />
+    </joint>
     <link name="lidar_frame_${lidar_prefix}">
       <collision>
@@ -64,114 +29,55 @@
       </collision>
       <visual>
+        <origin xyz="0 0 ${ld06_base_box_height / 2}" rpy="0 0 0" />
         <geometry>
           <box size="${ld06_base_box_width} ${ld06_base_box_width / 2} ${ld06_base_box_height}" />
         </geometry>
-        <origin xyz="0 0 0" rpy="0 0 0" />
         <material name="ld06_${lidar_prefix}_grey" />
       </visual>
-    </link>
-    <gazebo reference="ld06_frame_${lidar_prefix}">
-      <material>
-        Gazebo/Grey
-      </material>
-    </gazebo>
-    <link name="ld06_base_cylinder_${lidar_prefix}">
-      <collision>
+      <visual> <!-- box-->
+        <origin xyz="0 0.017 ${ld06_base_box_height + (ld06_box_height / 2)}" rpy="0 0 0" />
         <geometry>
-          <cylinder radius="${ld06_base_box_width / 2}" length="${ld06_base_box_height}" />
+          <box size="${ld06_box_width} ${ld06_box_width} ${ld06_box_height}" />
         </geometry>
-      </collision>
-      <visual>
+        <material name="ld06_${lidar_prefix}_blackish" />
+      </visual>
+      <visual> <!-- cylinder -->
+        <origin xyz="0 0.017 ${(ld06_base_box_height + ld06_box_height) +(ld06_cylinder_height / 2)}" rpy="0 0 0" />
+        <geometry>
+          <cylinder radius="${ld06_cylinder_radius}" length="${ld06_cylinder_height}" />
+        </geometry>
+        <material name="ld06_${lidar_prefix}_cylinder" />
+      </visual>
+      <visual> <!-- base_cylinder -->
         <geometry>
           <cylinder radius="${ld06_base_box_width / 2}" length="${ld06_base_box_height}" />
         </geometry>
         <material name="ld06_${lidar_prefix}_grey" />
-        <origin xyz="0 ${ld06_base_box_width / 4} 0" rpy="0 0 0" />
+        <origin xyz="0 ${ld06_base_box_width / 4} ${(ld06_base_box_height / 2)}" rpy="0 0 0" />
       </visual>
+     <xacro:solid_cuboid_inertial rpy="0 0 0" xyz="0 0 0" mass_kg="0.001" x="${ld06_base_box_width}" y="${ld06_base_box_width / 2}" z="${ld06_base_box_height}" />
     </link>
-    <gazebo reference="ld06_base_cylinder_${lidar_prefix}">
-      <material>
-        Gazebo/Grey
-      </material>
-    </gazebo>
-    <joint name="ld06_base_cylinder_base_box_${lidar_prefix}" type="fixed">
-      <parent link="lidar_frame_${lidar_prefix}" />
-      <child link="ld06_base_cylinder_${lidar_prefix}" />
-      <origin xyz="0 0 0" rpy="0 0 0" />
-      <axis xyz="0 0 0" />
-    </joint>
-    <joint name="ld06_box_base_box_${lidar_prefix}" type="fixed">
-      <parent link="lidar_frame_${lidar_prefix}" />
-      <child link="ld06_box_${lidar_prefix}" />
-      <origin xyz="0 0.017 ${ld06_base_box_height}" rpy="0 0 0" />
-      <axis xyz="0 0 0" />
-    </joint>
-    <joint name="ld06_cylinder_box_${lidar_prefix}" type="fixed">
-      <parent link="ld06_box_${lidar_prefix}" />
-      <child link="ld06_cylinder_${lidar_prefix}" />
-      <origin xyz="0 0 ${ld06_box_height - ld06_cylinder_height/2}" rpy="0 0 0" />
-      <axis xyz="0 0 0" />
-    </joint>
-    <!-- <joint name="base_to_lidar_frame_${lidar_prefix}" type="fixed">
-      <parent link="scan" />
-      <child link="lidar_frame_${lidar_prefix}" />
-      <origin xyz="0 0 0" rpy="0 0 -${M_PI / 2}" />
-    </joint> -->
-    <joint name="base_to_lidar_frame_${lidar_prefix}" type="fixed">
-      <parent link="base_link" />
-      <child link="lidar_frame_${lidar_prefix}" />
-      <xacro:insert_block name="joint_pose" />
-    </joint>
     <gazebo reference="lidar_frame_${lidar_prefix}">
       <material>Gazebo/Black</material>
-      <sensor name='gpu_lidar' type='gpu_lidar'>"
-        <pose relative_to='lidar_frame_${lidar_prefix}'>0 0 0 0 0 0</pose>
-        <topic>/scan</topic>
-        <gz_frame_id>lidar_frame_${lidar_prefix}</gz_frame_id>
-        <update_rate>10</update_rate>
-        <ray>
-            <scan>
-                <horizontal>
-                    <samples>450</samples>
-                    <resolution>1</resolution>
-                    <min_angle>-0</min_angle>
-                    <max_angle>6.28</max_angle>
-                </horizontal>
-                <vertical>
-                    <samples>1</samples>
-                    <resolution>0.01</resolution>
-                    <min_angle>0</min_angle>
-                    <max_angle>0</max_angle>
-                </vertical>
-            </scan>
-            <range>
-                <min>0.05</min>
-                <max>10.0</max>
-                <resolution>0.01</resolution>
-            </range>
-        </ray>
-        <always_on>1</always_on>
-        <visualize>true</visualize>
-    </sensor>
-    <!-- <sensor name="laser" type="gpu_lidar">
+      <sensor name="laser" type="gpu_lidar">
         <pose> 0 0 0 0 0 0 </pose>
-        <visualize>true</visualize>
+        <visualize>false</visualize>
         <update_rate>10</update_rate>
         <lidar>
           <scan>
             <horizontal>
-              <samples>450</samples>
-              <min_angle>0</min_angle>
-              <max_angle>6.28</max_angle>
+              <samples>360</samples>
+              <min_angle>-3.14</min_angle>
+              <max_angle>3.14</max_angle>
             </horizontal>
           </scan>
           <range>
-            <min>0.05</min>
-            <max>10.0</max>
+            <min>0.3</min>
+            <max>12</max>
           </range>
         </lidar>
-        <topic>/scan</topic>
+        <topic>scan</topic>
         <gz_frame_id>lidar_frame_${lidar_prefix}</gz_frame_id>
-      </sensor> -->
+      </sensor>
     </gazebo>
   </xacro:macro>

File: description/urdf/properties.urdf.xacro (robot description, xacro)
@@ -2,5 +2,5 @@
 <robot xmlns:xacro="http://ros.org/wiki/xacro">
   <xacro:property name="M_PI" value="3.14159" />
-  <xacro:property name="body_height" value="0.290" />
+  <xacro:property name="body_height" value="0.300" />
   <xacro:property name="body_radius" value="0.2286" />
   <xacro:property name="mass" value="22" />

Commit message: Fixed base_footprint->base_link offset. Corrected LIDAR position.

File: description/urdf/base.urdf.xacro (robot description, xacro)
@@ -48,5 +48,5 @@
   <link name="base_footprint" />
   <joint name="base_footprint_joint" type="fixed">
-    <origin xyz="0 0 ${base_to_floor_z_offset}" rpy="0 0 0" />
+    <origin xyz="0 0 -${base_to_floor_z_offset}" rpy="0 0 0" />
     <child link="base_footprint" />
     <parent link="base_link" />
