Commit message: Sigyn wheel macro much improved

File: description/urdf/sigyn_wheels_macro.urdf.xacro (robot description, xacro)
@@ -1,13 +1,15 @@
 <?xml version="1.0"?>
 <robot xmlns:xacro="http://ros.org/wiki/xacro">
-  <xacro:macro name="wheel" params="side radius width pos_x pos_y pos_z mass_kg">
-    <foo side="${side}" radius="${radius}" width="${width}" pos_x="${pos_x}" pos_y="${pos_y}" pos_z="${pos_z}" mass_kg="${mass_kg}"/>
+  <xacro:macro name="wheel" params="axis side radius width pos_x pos_y pos_z mass_kg">
+    <!-- Create the outer, rubber tire -->
     <link name="${side}_wheel_link">
-      <visual>
-        <origin xyz="0 0 0" rpy="${pi/2} 0 0" />
+      <visual name="tire">
+        <origin xyz="0 0 0" rpy="0 0 0" />
         <geometry>
-          <cylinder radius="${radius}" length="${width}" />
+          <cylinder radius="${radius}" length="${width - 0.004}" />
         </geometry>
-        <material name="wheel_material" />
+        <material name="wheel_black">
+          <color rgba="0.15 0.15 0.15 1.0" />
+        </material>
       </visual>
       <collision>
@@ -22,7 +24,7 @@
       <visual>
         <material>
-          <ambient>0.1764 0.4588 0.8509 1.0</ambient>
-          <diffuse>0.1764 0.4588 0.8509 1.0</diffuse>
-          <specular>0.1764 0.4588 0.8509 1.0</specular>
+          <ambient>0.15 0.15 0.15 1.0</ambient>
+          <diffuse>0.15 0.15 0.15 1.0</diffuse>
+          <specular>0.15 0.15 0.15 1.0</specular>
           <emissive>0.0 0.0 0.0 0.0</emissive>
         </material>
@@ -30,8 +32,63 @@
     </gazebo>
     <joint name="${side}_wheel_joint" type="continuous">
-      <axis xyz="0 1 0" />
+      <axis xyz="0 0 ${axis}" />
       <parent link="base_link" />
       <child link="${side}_wheel_link" />
-      <origin xyz="${pos_x} ${pos_y} ${pos_z}" rpy="0 0 0" />
+      <origin xyz="${pos_x} ${pos_y} ${pos_z}" rpy="${-axis * pi / 2} 0 0" />
+    </joint>
+    <!-- Create the wheel hub -->
+    <link name="${side}_wheel_hub">
+      <origin xyz="0 0 0" rpy="0 0 0" />
+      <visual>
+        <geometry>
+          <cylinder radius="${radius - 0.02}" length="${width - 0.002}" />
+        </geometry>
+        <material name="wheel_silver">
+          <color rgba="0.8 0.8 0.8 1.0" />
+        </material>
+      </visual>
+    </link>
+    <gazebo reference="${side}_wheel_hub">
+      <visual>
+        <material>
+          <ambient>0.8 0.8 0.8 1.0</ambient>
+          <diffuse>0.8 0.8 0.8 1.0</diffuse>
+          <specular>0.8 0.8 0.8 1.0</specular>
+          <emissive>0.0 0.0 0.0 0.0</emissive>
+        </material>
+      </visual>
+    </gazebo>
+    <joint name="${side}_wheel_hub_joint" type="fixed">
+      <axis xyz="0 0 ${axis}" />
+      <parent link="${side}_wheel_link" />
+      <child link="${side}_wheel_hub" />
+      <origin xyz="0 0 0" rpy="0 0 0" />
+    </joint>
+    <!-- Create the wheel marker -->
+    <link name="${side}_wheel_marker">
+      <origin xyz="0 0 0" rpy="0 0 0" />
+      <visual>
+        <geometry>
+          <box size="0.01 ${(radius / 2)} ${width}" />
+        </geometry>
+        <material name="wheel_marker">
+          <color rgba="0.86 0.54 0.86 1" />
+        </material>
+      </visual>
+    </link>
+    <gazebo reference="${side}_wheel_marker">
+      <visual>
+        <material>
+          <ambient>0.86 0.54 0.86 1.0</ambient>
+          <diffuse>0.86 0.54 0.86 1.0</diffuse>
+          <specular>0.86 0.54 0.86 1.0</specular>
+          <emissive>0.0 0.0 0.0 0.0</emissive>
+        </material>
+      </visual>
+    </gazebo>
+    <joint name="${side}_wheel_marker_joint" type="fixed">
+      <parent link="${side}_wheel_hub" />
+      <child link="${side}_wheel_marker" />
+      <origin xyz="0 ${(radius - 0.02) / 2} 0" rpy="0 0 0" />
     </joint>
   </xacro:macro>
@@ -43,11 +100,8 @@
       <xacro:property name="y" value="${(config.body.radius-config.wheels.center_offset)*instance['y_position_multiplier']}"/>
       <xacro:property name="z" value="-${(config.wheels.gear_box_height/2)+config.wheels.gear_box_spacing_from_base}"/>
-      <xacro:wheel pos_y="${y}" pos_z="${z}" side="${instance['name']}" radius="${config.wheels.radius}" width="${config.wheels.width}" pos_x="0.0" mass_kg="${config.wheels.mass}" />
+      <xacro:wheel axis="${instance['y_position_multiplier']}" pos_y="${y}" pos_z="${z}" side="${instance['name']}" radius="${config.wheels.radius}" width="${config.wheels.width}" pos_x="0.0" mass_kg="${config.wheels.mass}" />
       <xacro:wheels config="${config}" instances="${instances}"/>
     </xacro:if>
   </xacro:macro>
-  <material name="wheel_material">
-    <color rgba="0.15 0.15 0.15 1" />
-  </material>
   <!--
 Copyright (c) 2024 Michael Wimble
