Commit message: Added color macros

File: description/urdf/sigyn_caster_wheel_macro.urdf.xacro (robot description, xacro)
@@ -2,6 +2,8 @@
 <robot xmlns:xacro="http://ros.org/wiki/xacro">
   <xacro:macro name="caster_wheel_upright" params="config name y_offset_multiplier">
+    <xacro:property name="pi" value="3.14159265359" />
     <xacro:property name="chassis_bottom" value="${config.wheels.radius + (config.wheels.gear_box_height / 2) + config.wheels.gear_box_spacing_from_base}" />
     <xacro:property name="upright_width" value="0.01" />
+    <xacro:property name="cf_color" value="0.7 0.7 0.72 1.0" />
     <link name="caster_frame_${name}">
       <visual>
@@ -11,5 +13,5 @@
         </geometry>
         <material name="caster_upright_color">
-          <color rgba="0.7 0.7 0.72 1.0" />
+          <color rgba="${cf_color}" />
         </material>
       </visual>
@@ -18,7 +20,7 @@
       <visual>
         <material>
-          <ambient>0.7 0.7 0.72 1.0</ambient>
-          <diffuse>0.7 0.7 0.72 1.0</diffuse>
-          <specular>0.7 0.7 0.72 1.0</specular>
+          <ambient>${cf_color}</ambient>
+          <diffuse>${cf_color}</diffuse>
+          <specular>${cf_color}</specular>
           <emissive>0.0 0.0 0.0 0.0</emissive>
         </material>
@@ -32,8 +34,6 @@
   </xacro:macro>
   <xacro:macro name="caster_wheel" params="config">
-    <xacro:property name="caster_radius" value="0.025" />
-    <xacro:property name="caster_width" value="0.023" />
-    <xacro:property name="caster_offset" value="0.035" />
-    <xacro:property name="caster_wheel_x" value="${-(body_radius-caster_offset)}" />
+    <xacro:property name="pi" value="3.14159265359" />
+    <xacro:property name="cw_color" value="0.416 0.051 0.047 1.0" />
     <link name="caster_wheel_link">
       <visual>
@@ -43,5 +43,5 @@
         </geometry>
         <material name="red">
-          <color rgba="0.416 0.051 0.047 1.0" />
+          <color rgba="${cw_color}" />
         </material>
       </visual>
@@ -59,7 +59,7 @@
       <visual>
         <material>
-          <ambient>0.416 0.051 0.047  1.0</ambient>
-          <diffuse>0.416 0.051 0.047  1.0</diffuse>
-          <specular>0.416 0.051 0.047  1.0</specular>
+          <ambient>${cw_color}</ambient>
+          <diffuse>${cw_color}</diffuse>
+          <specular>${cw_color}</specular>
           <emissive>0.0 0.0 0.0 0.0</emissive>
         </material>

Commit message: Fix collision for gazebo

File: description/urdf/sigyn_caster_wheel_macro.urdf.xacro (robot description, xacro)
@@ -50,5 +50,5 @@
         </visual>
         <collision>
-          <origin xyz="0 0 0" rpy="${pi/2} 0 0" />
+          <origin xyz="0 0 0" rpy="0 0 0" />
           <geometry>
             <cylinder radius="${config.caster.radius}" length="${config.caster.width}" />

File: description/urdf/sigyn_wheels_macro.urdf.xacro (robot description, xacro)
@@ -31,7 +31,7 @@
         </visual>
         <collision>
-          <origin xyz="0 0 0" rpy="${pi/2} 0 0" />
+          <origin xyz="0 0 0" rpy="0 0 0" />
           <geometry>
-            <cylinder radius="${radius}" length="${width}" />
+            <cylinder radius="${radius}" length="${width - 0.004}" />
           </geometry>
         </collision>
