Commit message: Moved copyrights

File: description/urdf/gazebo.urdf.xacro (robot description, xacro)
@@ -1,20 +1,2 @@
-<!--
-Copyright (c) 2024 Michael Wimble
-Permission is hereby granted, free of charge, to any person obtaining a copy
-of this software and associated documentation files (the "Software"), to deal
-in the Software without restriction, including without limitation the rights
-to use, copy, modify, merge, publish, distribute, sublicense, and/or sell
-copies of the Software, and to permit persons to whom the Software is
-furnished to do so, subject to the following conditions:
-The above copyright notice and this permission notice shall be included in all
-copies or substantial portions of the Software.
-THE SOFTWARE IS PROVIDED "AS IS", WITHOUT WARRANTY OF ANY KIND, EXPRESS OR
-IMPLIED, INCLUDING BUT NOT LIMITED TO THE WARRANTIES OF MERCHANTABILITY,
-FITNESS FOR A PARTICULAR PURPOSE AND NONINFRINGEMENT. IN NO EVENT SHALL THE
-AUTHORS OR COPYRIGHT HOLDERS BE LIABLE FOR ANY CLAIM, DAMAGES OR OTHER
-LIABILITY, WHETHER IN AN ACTION OF CONTRACT, TORT OR OTHERWISE, ARISING FROM,
-OUT OF OR IN CONNECTION WITH THE SOFTWARE OR THE USE OR OTHER DEALINGS IN THE
-SOFTWARE.
--->
 <robot xmlns:xacro="http://ros.org/wiki/xacro">
   <xacro:macro name="diff_drive_controller" params="wheel_separation wheel_radius">
@@ -38,3 +20,21 @@
     </gazebo>
   </xacro:macro>
+  <!--
+Copyright (c) 2024 Michael Wimble
+Permission is hereby granted, free of charge, to any person obtaining a copy
+of this software and associated documentation files (the "Software"), to deal
+in the Software without restriction, including without limitation the rights
+to use, copy, modify, merge, publish, distribute, sublicense, and/or sell
+copies of the Software, and to permit persons to whom the Software is
+furnished to do so, subject to the following conditions:
+The above copyright notice and this permission notice shall be included in all
+copies or substantial portions of the Software.
+THE SOFTWARE IS PROVIDED "AS IS", WITHOUT WARRANTY OF ANY KIND, EXPRESS OR
+IMPLIED, INCLUDING BUT NOT LIMITED TO THE WARRANTIES OF MERCHANTABILITY,
+FITNESS FOR A PARTICULAR PURPOSE AND NONINFRINGEMENT. IN NO EVENT SHALL THE
+AUTHORS OR COPYRIGHT HOLDERS BE LIABLE FOR ANY CLAIM, DAMAGES OR OTHER
+LIABILITY, WHETHER IN AN ACTION OF CONTRACT, TORT OR OTHERWISE, ARISING FROM,
+OUT OF OR IN CONNECTION WITH THE SOFTWARE OR THE USE OR OTHER DEALINGS IN THE
+SOFTWARE.
+-->
 </robot>

File: description/urdf/ld06.urdf.xacro (robot description, xacro)
@@ -1,21 +1,3 @@
 <?xml version="1.0"?>
-<!--
-Copyright (c) 2024 Michael Wimble
-Permission is hereby granted, free of charge, to any person obtaining a copy
-of this software and associated documentation files (the "Software"), to deal
-in the Software without restriction, including without limitation the rights
-to use, copy, modify, merge, publish, distribute, sublicense, and/or sell
-copies of the Software, and to permit persons to whom the Software is
-furnished to do so, subject to the following conditions:
-The above copyright notice and this permission notice shall be included in all
-copies or substantial portions of the Software.
-THE SOFTWARE IS PROVIDED "AS IS", WITHOUT WARRANTY OF ANY KIND, EXPRESS OR
-IMPLIED, INCLUDING BUT NOT LIMITED TO THE WARRANTIES OF MERCHANTABILITY,
-FITNESS FOR A PARTICULAR PURPOSE AND NONINFRINGEMENT. IN NO EVENT SHALL THE
-AUTHORS OR COPYRIGHT HOLDERS BE LIABLE FOR ANY CLAIM, DAMAGES OR OTHER
-LIABILITY, WHETHER IN AN ACTION OF CONTRACT, TORT OR OTHERWISE, ARISING FROM,
-OUT OF OR IN CONNECTION WITH THE SOFTWARE OR THE USE OR OTHER DEALINGS IN THE
-SOFTWARE.
--->
 <robot xmlns:xacro="http://ros.org/wiki/xacro" name="ld06">
   <xacro:macro name="ld06" params="lidar_prefix *joint_pose">
@@ -178,3 +160,21 @@
     </gazebo>
   </xacro:macro>
+<!--
+Copyright (c) 2024 Michael Wimble
+Permission is hereby granted, free of charge, to any person obtaining a copy
+of this software and associated documentation files (the "Software"), to deal
+in the Software without restriction, including without limitation the rights
+to use, copy, modify, merge, publish, distribute, sublicense, and/or sell
+copies of the Software, and to permit persons to whom the Software is
+furnished to do so, subject to the following conditions:
+The above copyright notice and this permission notice shall be included in all
+copies or substantial portions of the Software.
+THE SOFTWARE IS PROVIDED "AS IS", WITHOUT WARRANTY OF ANY KIND, EXPRESS OR
+IMPLIED, INCLUDING BUT NOT LIMITED TO THE WARRANTIES OF MERCHANTABILITY,
+FITNESS FOR A PARTICULAR PURPOSE AND NONINFRINGEMENT. IN NO EVENT SHALL THE
+AUTHORS OR COPYRIGHT HOLDERS BE LIABLE FOR ANY CLAIM, DAMAGES OR OTHER
+LIABILITY, WHETHER IN AN ACTION OF CONTRACT, TORT OR OTHERWISE, ARISING FROM,
+OUT OF OR IN CONNECTION WITH THE SOFTWARE OR THE USE OR OTHER DEALINGS IN THE
+SOFTWARE.
+-->
 </robot>

File: description/urdf/material.urdf.xacro (robot description, xacro)
@@ -1,3 +1,16 @@
 <?xml version="1.0"?>
+<robot xmlns:xacro="http://ros.org/wiki/xacro" name="material">
+    <material name="aluminum_frame">
+        <color rgba="0.516 0.527 0.535 1" />
+    </material>
+    <material name="caster_wheel_material">
+        <color rgba="0.9 0.1 0.1 1" />
+    </material>
+    <material name="t265_material">
+        <color rgba="0.80 0.40 0.60 1" />
+    </material>
+    <material name="wheel_material">
+        <color rgba="0.15 0.15 0.15 1" />
+    </material>
 <!--
 Copyright (c) 2024 Michael Wimble
@@ -18,16 +31,3 @@
 SOFTWARE.
 -->
-<robot xmlns:xacro="http://ros.org/wiki/xacro" name="material">
-    <material name="aluminum_frame">
-        <color rgba="0.516 0.527 0.535 1" />
-    </material>
-    <material name="caster_wheel_material">
-        <color rgba="0.9 0.1 0.1 1" />
-    </material>
-    <material name="t265_material">
-        <color rgba="0.80 0.40 0.60 1" />
-    </material>
-    <material name="wheel_material">
-        <color rgba="0.15 0.15 0.15 1" />
-    </material>
 </robot>

Commit message: Cleanup, more iteration macros for gazebo

File: description/urdf/gazebo.urdf.xacro (robot description, xacro)
@@ -1,32 +1,3 @@
-<robot xmlns:xacro="http://ros.org/wiki/xacro">
-  <xacro:macro name="diff_drive_controller" params="wheel_separation wheel_radius">
-    <gazebo>
-      <plugin name="gz::sim::systems::DiffDrive" filename="gz-sim-diff-drive-system">
-        <!-- Wheel Information -->
-        <left_joint>left_wheel_joint</left_joint>
-        <right_joint>right_wheel_joint</right_joint>
-        <wheel_separation>${wheel_separation}</wheel_separation>
-        <wheel_radius>${wheel_radius}</wheel_radius>
-        <!-- Limits -->
-        <!-- <max_wheel_torque>200</max_wheel_torque> -->
-        <max_linear_acceleration>1.0</max_linear_acceleration>
-        <!-- Input -->
-        <topic>cmd_vel</topic>
-        <!-- Output -->
-        <frame_id>odom</frame_id>
-        <child_frame_id>base_link</child_frame_id>
-        <odom_topic>odom</odom_topic>
-        <odom_publisher_frequency>30</odom_publisher_frequency>
-        <tf_topic>/tf</tf_topic>
-      </plugin>
-      <plugin filename="gz-sim-joint-state-publisher-system"
-        name="gz::sim::systems::JointStatePublisher">
-        <topic>joint_states</topic>
-        <joint_name>left_wheel_joint</joint_name>
-        <joint_name>right_wheel_joint</joint_name>
-      </plugin>
-    </gazebo>
-  </xacro:macro>
-  <!--
+<!--
 Copyright (c) 2024 Michael Wimble
 Permission is hereby granted, free of charge, to any person obtaining a copy
@@ -46,3 +17,43 @@
 SOFTWARE.
 -->
+<robot xmlns:xacro="http://ros.org/wiki/xacro">
+  <xacro:macro name="gazebo_wheels" params="instances:=^*">
+    <xacro:if value="${instances}">
+      <xacro:property name="instance" value="${instances.pop(0)}"/>
+      <xacro:element xacro:name="${instance['name']}_joint">${instance['name']}_wheel_joint</xacro:element>
+      <xacro:gazebo_wheels instances="${instances}"/>
+    </xacro:if>
+  </xacro:macro>
+  <xacro:macro name="gazebo_joints" params="instances:=^*">
+    <xacro:if value="${instances}">
+      <xacro:property name="instance" value="${instances.pop(0)}"/>
+      <joint_name>${instance['name']}wheel__joint</joint_name>
+      <xacro:gazebo_joints instances="${instances}"/>
+    </xacro:if>
+  </xacro:macro>
+  <xacro:macro name="diff_drive_controller" params="config instances1 instances2">
+    <gazebo>
+      <plugin name="gz::sim::systems::DiffDrive" filename="gz-sim-diff-drive-system">
+        <!-- Wheel Information -->
+        <xacro:gazebo_wheels instances="${instances1}"/>
+        <wheel_separation>${(config.body.radius - config.wheels.center_offset) * 2}</wheel_separation>
+        <wheel_radius>${config.wheels.radius}</wheel_radius>
+        <!-- Limits -->
+        <!-- <max_wheel_torque>200</max_wheel_torque> -->
+        <max_linear_acceleration>1.0</max_linear_acceleration>
+        <!-- Input -->
+        <topic>cmd_vel</topic>
+        <!-- Output -->
+        <frame_id>odom</frame_id>
+        <child_frame_id>base_footprint</child_frame_id>
+        <odom_topic>odom</odom_topic>
+        <odom_publisher_frequency>30</odom_publisher_frequency>
+        <tf_topic>/tf</tf_topic>
+      </plugin>
+      <plugin filename="gz-sim-joint-state-publisher-system" name="gz::sim::systems::JointStatePublisher">
+        <topic>joint_states</topic>
+        <xacro:gazebo_joints instances="${instances2}"/>
+      </plugin>
+    </gazebo>
+  </xacro:macro>
 </robot>

File: description/urdf/sigyn.urdf.xacro (robot description, xacro)
@@ -9,10 +9,4 @@
   <xacro:arg name="use_ros2_control" default="true" />
   <xacro:arg name="sim_mode" default="false" />
-  <xacro:if value="$(arg use_ros2_control)">
-    <xacro:include filename="ros2_control.xacro" />
-  </xacro:if>
-  <xacro:unless value="$(arg use_ros2_control)">
-    <xacro:include filename="gazebo_control.xacro" />
-  </xacro:unless>
   <!-- Make the body-->
   <xacro:sigyn_base body_props="${props.body}" wheels_props="${props.wheels}" />
@@ -21,5 +15,4 @@
   <!-- Make the caster wheel -->
   <xacro:caster_wheel config="${props}" />
-  <xacro:include filename="$(find description)/urdf/properties.urdf.xacro" />
   <xacro:include filename="$(find description)/urdf/ld06.urdf.xacro" />
   <xacro:include filename="$(find description)/urdf/gazebo.urdf.xacro" />
@@ -27,4 +20,4 @@
     <origin xyz="0.155 0 0.300" rpy="0 0 -${pi / 2}" />
   </xacro:ld06>
-  <xacro:diff_drive_controller wheel_separation="${wheel_pos_y * 2}" wheel_radius="${wheel_radius}" />
+  <xacro:diff_drive_controller config="${props}" instances1="${props.wheels.instances}" instances2="${props.wheels.instances}" />
 </robot>

Commit message: Fix for base_footprint

File: description/urdf/gazebo.urdf.xacro (robot description, xacro)
@@ -46,5 +46,5 @@
         <!-- Output -->
         <frame_id>odom</frame_id>
-        <child_frame_id>base_footprint</child_frame_id>
+        <child_frame_id>base_link</child_frame_id>
         <odom_topic>odom</odom_topic>
         <odom_publisher_frequency>50</odom_publisher_frequency>

File: description/urdf/sigyn_base_macro.urdf.xacro (robot description, xacro)
@@ -29,6 +29,6 @@
     <joint name="base_footprint_to_base_link" type="fixed">
       <origin xyz="0 0 -${wheels_props.radius + (wheels_props.gear_box_height / 2) + wheels_props.gear_box_spacing_from_base}" rpy="0 0 0" />
-      <parent link="base_footprint" />
-      <child link="base_link" />
+      <child link="base_footprint" />
+      <parent link="base_link" />
     </joint>
     <material name="body_aluminum">

Commit message: Start of pi_servo1

File: description/urdf/gazebo.urdf.xacro (robot description, xacro)
@@ -54,4 +54,5 @@
         <topic>joint_states</topic>
         <xacro:gazebo_joints instances="${instances2}"/>
+        <joint_name>servo1_joint</joint_name>
       </plugin>
         <!-- GROUND ODOMETRY POSITION STATE PUBLISHER (FAKE LOCALIZATION) -->

File: description/urdf/ros2_control.xacro (robot description, xacro)
@@ -2,4 +2,19 @@
 <robot xmlns:xacro="http://www.ros.org/wiki/xacro">
   <xacro:unless value="$(arg sim_mode)">
+    <ros2_control name="endgripper_servo" type="actuator">
+      <hardware>
+        <plugin>pi_servo1/EndGripperJoint</plugin>
+        <param name="example_param_hw_start_duration_sec">2.0</param>
+        <param name="example_param_hw_stop_duration_sec">3.0</param>
+        <param name="example_param_hw_slowdown">1.23</param>
+      </hardware>
+      <joint name="servo1_joint">
+        <command_interface name="position">
+          <param name="min">-100</param>
+          <param name="max">100</param>
+        </command_interface>
+        <state_interface name="position"/>
+      </joint>
+    </ros2_control>
     <ros2_control name="RealRobot" type="system">
       <hardware>
@@ -32,4 +47,19 @@
   </xacro:unless>
   <xacro:if value="$(arg sim_mode)">
+    <!-- <ros2_control name="endgripper_servo" type="actuator">
+      <hardware>
+        <plugin>pi_servo1/EndGripperJoint</plugin>
+        <param name="example_param_hw_start_duration_sec">2.0</param>
+        <param name="example_param_hw_stop_duration_sec">3.0</param>
+        <param name="example_param_hw_slowdown">1.23</param>
+      </hardware>
+      <joint name="servo1_joint">
+        <command_interface name="position">
+          <param name="min">-100</param>
+          <param name="max">100</param>
+        </command_interface>
+        <state_interface name="position"/>
+      </joint>
+    </ros2_control> -->
     <ros2_control name="GazeboSystem" type="system">
       <hardware>
@@ -52,4 +82,11 @@
         <state_interface name="position" />
       </joint>
+      <joint name="servo1_joint">
+        <command_interface name="position">
+          <param name="min">-100</param>
+          <param name="max">100</param>
+        </command_interface>
+        <state_interface name="position"/>
+      </joint>
     </ros2_control>
   </xacro:if>

File: description/urdf/sigyn.urdf.xacro (robot description, xacro)
@@ -29,4 +29,53 @@
     <origin xyz="0.155 0 0.300" rpy="0 0 -${pi / 2}" />
   </xacro:ld06>
+  <material name="red">
+    <color rgba="0.8 0.0 0.0 1.0"/>
+  </material>
+  <joint name="servo1_joint" type="continuous">
+    <parent link="base_link" />
+    <child link="servo1" />
+    <origin xyz="0.0 0.0 1.0" rpy="0 0 0" />
+    <axis xyz="0 1 0"/>
+    <dynamics damping="0.7"/>
+    <limit lower="-10" upper="10" effort="100" velocity="1.0"/>
+    <material name="red">
+      <color rgba="0.8 0.0 0.0 1.0"/>
+    </material>
+  </joint>
+  <link name="servo1">
+    <inertial>
+      <origin xyz="0 0 0" />
+      <mass value="0.1" />
+      <inertia ixx="0.0001" ixy="0.0" ixz="0.0" iyy="0.0001" iyz="0.0" izz="0.0001" />
+    </inertial>
+    <visual>
+      <origin xyz="0 0 1" />
+      <geometry>
+        <cylinder radius="0.05" length="0.2" />
+      </geometry>
+      <material name="red" />
+    </visual>
+    <collision>
+      <origin xyz="0 0 1" />
+      <geometry>
+        <cylinder radius="0.05" length="0.2" />
+      </geometry>
+    </collision>
+  </link>
+  <gazebo>
+    <plugin filename="gz-sim-joint-position-controller-system" name="gz::sim::systems::JointPositionController">
+      <joint_name>servo1_joint</joint_name>
+      <!-- <sub_topic>servo1</sub_topic> -->
+      <p_gain>1.0</p_gain>
+      <i_gain>0.0</i_gain>
+      <d_gain>0.0</d_gain>
+      <i_max>0.0</i_max>
+      <i_min>0.0</i_min>
+      <cmd_max>1</cmd_max>
+      <cmd_min>-1</cmd_min>
+      <!-- <type>COMMAND</type> -->
+      <topic>/servo1/position</topic>
+    </plugin>
+  </gazebo>
   <xacro:diff_drive_controller config="${props}" instances1="${props.wheels.instances}" instances2="${props.wheels.instances}" />
 </robot>
