Commit message: Snapshot, gazebo pole connector_plate working

File: description/urdf/gazebo.urdf.xacro (robot description, xacro)
@@ -54,5 +54,5 @@
         <topic>joint_states</topic>
         <xacro:gazebo_joints instances="${instances2}"/>
-        <joint_name>servo1_joint</joint_name>
+        <joint_name>elevator_pole_to_elevator_connector_plate</joint_name>
       </plugin>
         <!-- GROUND ODOMETRY POSITION STATE PUBLISHER (FAKE LOCALIZATION) -->

File: description/urdf/gripper_assembly.urdf.xacro (robot description, xacro)
@@ -2,149 +2,170 @@
 <robot xmlns:xacro="http://ros.org/wiki/xacro" name="Sigyn">
     <xacro:include filename="$(find description)/urdf/gripper_assembly_properties.urdf.xacro" />
-    <link name="evalator_pole">
-        <visual>
-            <geometry>
-                <box size="${elevator_pole_length} ${elevator_pole_width} ${elevator_pole_height}" />
-            </geometry>
-            <material name="evalator_pole_color">
-                <color rgba="0.8 0.8 0.8 0.7" />
-            </material>
-        </visual>
-    </link>
-    <link name="conveyor belt">
-        <visual>
-            <geometry>
-                <box size="${elevator_pole_length} 0.02 ${elevator_pole_height}" />
-            </geometry>
-            <material name="evalator_pole_belt_color">
-                <color rgba="0.0 0.0 0.0 1.0" />
-            </material>
-            <origin xyz="0.0 0.001 0.0" rpy="0 0 ${pi/2}" />
-        </visual>
-    </link>
+    <xacro:colorize_link color="0.95 1.0 0.95 1.0" name="evelator_pole">
+        <foo>
+            <visual>
+                <geometry>
+                    <box size="${elevator_pole_length} ${elevator_pole_width} ${elevator_pole_height}" />
+                </geometry>
+                <material name="evelator_pole"/>
+            </visual>
+            <collision>
+                <geometry>
+                    <box size="${elevator_pole_length} ${elevator_pole_width} ${elevator_pole_height}" />
+                </geometry>
+            </collision>
+            <xacro:solid_cuboid_inertial rpy="0 0 0" xyz="0 0 0" mass_kg="0.1" x="${elevator_pole_length}" y="${elevator_pole_width}" z="${elevator_pole_height}" />
+        </foo>
+    </xacro:colorize_link>
+    <xacro:colorize_link color="0.2 0.2 0.2 1.0" name="conveyor_belt">
+        <foo>
+            <visual>
+                <geometry>
+                    <box size="0.02 0.001 ${elevator_pole_height}" />
+                </geometry>
+                <material name="conveyor_belt"/>
+            </visual>
+            <collision>
+                <geometry>
+                    <box size="0.02 0.001 ${elevator_pole_height}" />
+                </geometry>
+            </collision>
+            <xacro:solid_cuboid_inertial rpy="0 0 0" xyz="0 0 0" mass_kg="0.01" x="${elevator_pole_length}" y="${elevator_pole_width}" z="${elevator_pole_height}" />
+        </foo>
+    </xacro:colorize_link>
     <joint name="elevator_pole_to_conveyor_belt" type="fixed">
-        <origin xyz="0.0 0.0 0.0" rpy="0 0 0" />
-        <parent link="evalator_pole" />
-        <child link="conveyor belt" />
+        <origin xyz="0.0 ${((elevator_pole_width/2)+0.0005)} 0.0" rpy="0 0 0" />
+        <parent link="evelator_pole" />
+        <child link="conveyor_belt" />
         <axis xyz="0 0 1" />
     </joint>
-    <joint name="evalator_pole_to_elevator_connector_plate" type="prismatic">
+    <xacro:colorize_link color="0.1 0.1 0.2 1" name="elevator_connector_plate">
+        <foo>
+            <visual>
+                <geometry>
+                    <box size="${elevator_connector_plate_length} ${elevator_connector_plate_height} ${elevator_connector_plate_width}" />
+                </geometry>
+                <material name="elevator_connector_plate_color">
+                    <color rgba="0.1 0.1 0.2 1" />
+                </material>
+            </visual>
+            <collision>
+                <geometry>
+                    <box size="${elevator_connector_plate_length} ${elevator_connector_plate_height} ${elevator_connector_plate_width}" />
+                </geometry>
+            </collision>
+            <xacro:solid_cuboid_inertial rpy="0 0 0" xyz="0 0 0" mass_kg="0.01" x="${elevator_connector_plate_length}" y="${elevator_connector_plate_height}" z="${elevator_connector_plate_width}" />
+        </foo>
+    </xacro:colorize_link>
+    <joint name="elevator_pole_to_elevator_connector_plate" type="prismatic">
         <origin xyz="0.0 ${(elevator_pole_width/2)+(elevator_connector_plate_height/2)} ${(-elevator_pole_height/2)+(elevator_connector_plate_width/2)}" rpy="0 0 0" />
+        <parent link="evelator_pole" />
         <child link="elevator_connector_plate" />
-        <parent link="evalator_pole" />
         <limit lower="0.15" upper="${elevator_pole_height-(elevator_connector_plate_width)}" effort="1" velocity="0.5" />
         <axis xyz="0 0 1" />
+        <dynamics damping="0.7"/>
     </joint>
-    <link name="elevator_connector_plate">
-        <visual>
-            <geometry>
-                <box size="${elevator_connector_plate_length} ${elevator_connector_plate_height} ${elevator_connector_plate_width}" />
-            </geometry>
-            <material name="elevator_connector_plate_color">
-                <color rgba="0.1 0.1 0.2 1" />
-            </material>
-        </visual>
-    </link>
-    <joint name="elevator_connector_plate_to_gripper_elevator_plate" type="fixed">
-        <origin xyz="${(gripper_elevator_plate_length/2)-(elevator_connector_plate_length/2)-elevator_connector_x_offset_from_end} ${(gripper_elevator_plate_height/2)+(elevator_connector_plate_height/2)} 0.0" rpy="0 0 0" />
-        <parent link="elevator_connector_plate" />
-        <child link="gripper_extender_base_plate" />
-        <axis xyz="1 0 0" />
-    </joint>
-    <link name="gripper_extender_base_plate">
-        <visual>
-            <geometry>
-                <box size="${gripper_elevator_plate_length} ${gripper_elevator_plate_height} ${gripper_elevator_plate_width}" />
-            </geometry>
-            <material name="gripper_elevator_plate_color">
-                <color rgba="0.2 0.3 0.2 1" />
-            </material>
-        </visual>
-    </link>
-    <joint name="gripper_elevator_plate_to_gripper_extender" type="prismatic">
-        <origin xyz="0.0 ${(gripper_extender_width/2) + (gripper_elevator_plate_height/2)} 0.0" rpy="0 0 0" />
-        <parent link="gripper_extender_base_plate" />
-        <child link="gripper_extender" />
-        <limit lower="0" upper="${gripper_elevator_plate_length}" effort="1" velocity="0.5" />
-        <axis xyz="1 0 0" />
-    </joint>
-    <link name="gripper_extender">
-        <visual>
-            <geometry>
-                <box size="${gripper_extender_length} ${gripper_extender_width} ${gripper_extender_height}" />
-            </geometry>
-            <material name="gripper_extender_color">
-                <color rgba="0.35 0.3 0.35 1" />
-            </material>
-        </visual>
-    </link>
-    <link name="gripper_wrist_servo">
-        <visual>
-            <geometry>
-                <box size="${gripper_wrist_length} ${gripper_wrist_width} ${gripper_wrist_depth}" />
-            </geometry>
-            <material name="gripper_wrist_servo_color">
-                <color rgba="0.0 0.05 0.05 1.0" />
-            </material>
-        </visual>
-    </link>
-    <joint name="gripper_exender_to_gripper_wrist" type="fixed">
-        <origin xyz="${(gripper_extender_length/2)+(gripper_wrist_length/2)} 0.0 0.0" rpy="${pi/2} 0 0" />
-        <parent link="gripper_extender" />
-        <child link="gripper_wrist_servo" />
-        <axis xyz="0 0 1" />
-    </joint>
-    <joint name="gripper_wrist_to_parallel_gripper_base_plate" type="revolute">
-        <origin xyz="${(gripper_wrist_length/2)+(parallel_gripper_base_plate_depth/2)} 0.0 0.0" rpy="0 ${pi/2} 0" />
-        <parent link="gripper_wrist_servo" />
-        <child link="parallel_gripper_base_plate" />
-        <limit lower="-1.57" upper="1.57" effort="1" velocity="0.5" />
-        <axis xyz="0 0 1" />
-    </joint>
-    <link name="parallel_gripper_base_plate">
-        <visual>
-            <origin xyz="0 0 0" rpy="0 0 0" />
-            <geometry>
-                <box size="${parallel_gripper_base_plate_length} ${parallel_gripper_base_plate_width} ${parallel_gripper_base_plate_depth}"/>
-            </geometry>
-            <material name="parallel_gripper_base_plate_color">
-                <color rgba="${66/255} ${55/255} ${7/255} 1.0" />
-            </material>
-        </visual>
-    </link>
-    <link name="left_finger">
-        <visual>
-            <geometry>
-                <box size="${finger_length} ${finger_width} ${finger_depth}" />
-            </geometry>
-            <material name="left_finger_color">
-                <color rgba="${15/255} ${20/255} ${57/255} 1.0" />
-            </material>
-        </visual>
-    </link>
-    <joint name="parallel_gripper_base_plate_to_left_finger" type="prismatic">
-        <origin xyz="${(parallel_gripper_base_plate_length/2) - (finger_depth/2)} 0 ${(parallel_gripper_base_plate_depth/2) + (finger_length/2)}" rpy="0 ${pi/2} 0" />
-        <parent link="parallel_gripper_base_plate" />
-        <child link="left_finger" />
-        <limit lower="-${(parallel_gripper_base_plate_length/2) - (finger_depth)}" upper="0" effort="1" velocity="0.5" />
-        <axis xyz="0 0 1" />
-    </joint>
-    <link name="right_finger">
-        <visual>
-            <geometry>
-                <box size="${finger_length} ${finger_width} ${finger_depth}" />
-            </geometry>
-            <material name="right_finger_color">
-                <color rgba="${69/255} ${16/255} ${29/255} 1.0" />
-            </material>
-        </visual>
-    </link>
-    <joint name="parallel_gripper_base_plate_to_right_finger" type="prismatic">
-        <origin xyz="${-(parallel_gripper_base_plate_length/2) + (finger_depth/2)} 0 ${(parallel_gripper_base_plate_depth/2) + (finger_length/2)}" rpy="0 ${pi/2} 0" />
-        <parent link="parallel_gripper_base_plate" />
-        <child link="right_finger" />
-        <limit lower="0" upper="${(parallel_gripper_base_plate_length/2) - (finger_depth)}" effort="1" velocity="0.5" />
-        <mimic joint="parallel_gripper_base_plate_to_left_finger" multiplier="-1" offset="0" />
-        <axis xyz="0 0 1" />
-    </joint>
+    <!--
+        <joint name="elevator_connector_plate_to_gripper_elevator_plate" type="fixed">
+            <origin xyz="${(gripper_elevator_plate_length/2)-(elevator_connector_plate_length/2)-elevator_connector_x_offset_from_end} ${(gripper_elevator_plate_height/2)+(elevator_connector_plate_height/2)} 0.0" rpy="0 0 0" />
+            <parent link="elevator_connector_plate" />
+            <child link="gripper_extender_base_plate" />
+            <axis xyz="1 0 0" />
+        </joint>
+        <link name="gripper_extender_base_plate">
+            <visual>
+                <geometry>
+                    <box size="${gripper_elevator_plate_length} ${gripper_elevator_plate_height} ${gripper_elevator_plate_width}" />
+                </geometry>
+                <material name="gripper_elevator_plate_color">
+                    <color rgba="0.2 0.3 0.2 1" />
+                </material>
+            </visual>
+        </link>
+        <joint name="gripper_elevator_plate_to_gripper_extender" type="prismatic">
+            <origin xyz="0.0 ${(gripper_extender_width/2) + (gripper_elevator_plate_height/2)} 0.0" rpy="0 0 0" />
+            <parent link="gripper_extender_base_plate" />
+            <child link="gripper_extender" />
+            <limit lower="0" upper="${gripper_elevator_plate_length}" effort="1" velocity="0.5" />
+            <axis xyz="1 0 0" />
+        </joint>
+        <link name="gripper_extender">
+            <visual>
+                <geometry>
+                    <box size="${gripper_extender_length} ${gripper_extender_width} ${gripper_extender_height}" />
+                </geometry>
+                <material name="gripper_extender_color">
+                    <color rgba="0.35 0.3 0.35 1" />
+                </material>
+            </visual>
+        </link>
+        <link name="gripper_wrist_servo">
+            <visual>
+                <geometry>
+                    <box size="${gripper_wrist_length} ${gripper_wrist_width} ${gripper_wrist_depth}" />
+                </geometry>
+                <material name="gripper_wrist_servo_color">
+                    <color rgba="0.0 0.05 0.05 1.0" />
+                </material>
+            </visual>
+        </link>
+        <joint name="gripper_exender_to_gripper_wrist" type="fixed">
+            <origin xyz="${(gripper_extender_length/2)+(gripper_wrist_length/2)} 0.0 0.0" rpy="${pi/2} 0 0" />
+            <parent link="gripper_extender" />
+            <child link="gripper_wrist_servo" />
+            <axis xyz="0 0 1" />
+        </joint>
+        <joint name="gripper_wrist_to_parallel_gripper_base_plate" type="revolute">
+            <origin xyz="${(gripper_wrist_length/2)+(parallel_gripper_base_plate_depth/2)} 0.0 0.0" rpy="0 ${pi/2} 0" />
+            <parent link="gripper_wrist_servo" />
+            <child link="parallel_gripper_base_plate" />
+            <limit lower="-1.57" upper="1.57" effort="1" velocity="0.5" />
+            <axis xyz="0 0 1" />
+        </joint>
+        <link name="parallel_gripper_base_plate">
+            <visual>
+                <origin xyz="0 0 0" rpy="0 0 0" />
+                <geometry>
+                    <box size="${parallel_gripper_base_plate_length} ${parallel_gripper_base_plate_width} ${parallel_gripper_base_plate_depth}"/>
+                </geometry>
+                <material name="parallel_gripper_base_plate_color">
+                    <color rgba="${66/255} ${55/255} ${7/255} 1.0" />
+                </material>
+            </visual>
+        </link>
+        <link name="left_finger">
+            <visual>
+                <geometry>
+                    <box size="${finger_length} ${finger_width} ${finger_depth}" />
+                </geometry>
+                <material name="left_finger_color">
+                    <color rgba="${15/255} ${20/255} ${57/255} 1.0" />
+                </material>
+            </visual>
+        </link>
+        <joint name="parallel_gripper_base_plate_to_left_finger" type="prismatic">
+            <origin xyz="${(parallel_gripper_base_plate_length/2) - (finger_depth/2)} 0 ${(parallel_gripper_base_plate_depth/2) + (finger_length/2)}" rpy="0 ${pi/2} 0" />
+            <parent link="parallel_gripper_base_plate" />
+            <child link="left_finger" />
+            <limit lower="-${(parallel_gripper_base_plate_length/2) - (finger_depth)}" upper="0" effort="1" velocity="0.5" />
+            <axis xyz="0 0 1" />
+        </joint>
+        <link name="right_finger">
+            <visual>
+                <geometry>
+                    <box size="${finger_length} ${finger_width} ${finger_depth}" />
+                </geometry>
+                <material name="right_finger_color">
+                    <color rgba="${69/255} ${16/255} ${29/255} 1.0" />
+                </material>
+            </visual>
+        </link>
+        <joint name="parallel_gripper_base_plate_to_right_finger" type="prismatic">
+            <origin xyz="${-(parallel_gripper_base_plate_length/2) + (finger_depth/2)} 0 ${(parallel_gripper_base_plate_depth/2) + (finger_length/2)}" rpy="0 ${pi/2} 0" />
+            <parent link="parallel_gripper_base_plate" />
+            <child link="right_finger" />
+            <limit lower="0" upper="${(parallel_gripper_base_plate_length/2) - (finger_depth)}" effort="1" velocity="0.5" />
+            <mimic joint="parallel_gripper_base_plate_to_left_finger" multiplier="-1" offset="0" />
+            <axis xyz="0 0 1" />
+        </joint> -->
 </robot>

File: description/urdf/gripper_assembly_properties.urdf.xacro (robot description, xacro)
@@ -1,5 +1,4 @@
 <?xml version="1.0"?>
 <robot xmlns:xacro="http://ros.org/wiki/xacro">
-    <xacro:property name="pi" value="3.14159" />
     <xacro:property name="elevator_pole_length" value="0.045" />
     <xacro:property name="elevator_pole_width" value="0.04" />

File: description/urdf/ros2_control.xacro (robot description, xacro)
@@ -54,8 +54,8 @@
         <param name="example_param_hw_slowdown">1.23</param>
       </hardware>
-      <joint name="servo1_joint">
+      <joint name="elevator_pole_to_elevator_connector_plate">
         <command_interface name="position">
-          <param name="min">-100</param>
-          <param name="max">100</param>
+          <param name="min">0.15</param>
+          <param name="max">1.355</param>
         </command_interface>
         <state_interface name="position"/>
@@ -82,5 +82,5 @@
         <state_interface name="position" />
       </joint>
-      <joint name="servo1_joint">
+      <joint name="elevator_pole_to_elevator_connector_plate">
         <command_interface name="position">
           <param name="min">-100</param>

File: description/urdf/sigyn.urdf.xacro (robot description, xacro)
@@ -29,41 +29,13 @@
     <origin xyz="0.155 0 0.300" rpy="0 0 -${pi / 2}" />
   </xacro:ld06>
-  <material name="red">
-    <color rgba="0.8 0.0 0.0 1.0"/>
-  </material>
-  <joint name="servo1_joint" type="continuous">
+  <xacro:include filename="$(find description)/urdf/gripper_assembly.urdf.xacro" />
+  <joint name="base_link_to_elevator_pole" type="fixed">
+    <origin xyz="-0.16 0.015 ${0.3 + (elevator_pole_height/2)}" rpy="0 0 0" />
     <parent link="base_link" />
-    <child link="servo1" />
-    <origin xyz="0.0 0.0 1.0" rpy="0 0 0" />
-    <axis xyz="0 1 0"/>
-    <dynamics damping="0.7"/>
-    <limit lower="-10" upper="10" effort="100" velocity="1.0"/>
-    <material name="red">
-      <color rgba="0.8 0.0 0.0 1.0"/>
-    </material>
+    <child link="evelator_pole" />
   </joint>
-  <link name="servo1">
-    <inertial>
-      <origin xyz="0 0 0" />
-      <mass value="0.1" />
-      <inertia ixx="0.0001" ixy="0.0" ixz="0.0" iyy="0.0001" iyz="0.0" izz="0.0001" />
-    </inertial>
-    <visual>
-      <origin xyz="0 0 1" />
-      <geometry>
-        <cylinder radius="0.05" length="0.2" />
-      </geometry>
-      <material name="red" />
-    </visual>
-    <collision>
-      <origin xyz="0 0 1" />
-      <geometry>
-        <cylinder radius="0.05" length="0.2" />
-      </geometry>
-    </collision>
-  </link>
   <gazebo>
     <plugin filename="gz-sim-joint-position-controller-system" name="gz::sim::systems::JointPositionController">
-      <joint_name>servo1_joint</joint_name>
+      <joint_name>elevator_pole_to_elevator_connector_plate</joint_name>
       <!-- <sub_topic>servo1</sub_topic> -->
       <p_gain>1.0</p_gain>
@@ -75,5 +47,5 @@
       <cmd_min>-1</cmd_min>
       <!-- <type>COMMAND</type> -->
-      <topic>/servo1/position</topic>
+      <topic>/elevator_connector_plate/position</topic>
     </plugin>
   </gazebo>
