Commit message: More improvements to gazebo lidar

File: description/urdf/ld06.urdf.xacro (robot description, xacro)
@@ -43,5 +43,7 @@
       </visual>
       <visual> <!-- cylinder -->
-        <origin xyz="0 0.017 ${(ld06_base_box_height + ld06_box_height) +(ld06_cylinder_height / 2)}" rpy="0 0 0" />
+        <origin
+          xyz="0 0.017 ${(ld06_base_box_height + ld06_box_height) +(ld06_cylinder_height / 2)}"
+          rpy="0 0 0" />
         <geometry>
           <cylinder radius="${ld06_cylinder_radius}" length="${ld06_cylinder_height}" />
@@ -56,11 +58,18 @@
         <origin xyz="0 ${ld06_base_box_width / 4} ${(ld06_base_box_height / 2)}" rpy="0 0 0" />
       </visual>
-     <xacro:solid_cuboid_inertial rpy="0 0 0" xyz="0 0 0" mass_kg="0.001" x="${ld06_base_box_width}" y="${ld06_base_box_width / 2}" z="${ld06_base_box_height}" />
+      <xacro:solid_cuboid_inertial rpy="0 0 0" xyz="0 0 0" mass_kg="0.001"
+        x="${ld06_base_box_width}" y="${ld06_base_box_width / 2}" z="${ld06_base_box_height}" />
     </link>
+    <link name="lidar_beam_${lidar_prefix}"></link>
+    <joint name="laser_beam_joint" type="fixed">
+      <parent link="lidar_frame_${lidar_prefix}" />
+      <child link="lidar_beam_${lidar_prefix}" />
+      <origin xyz="0 0 0.04" rpy="0 0 0" />
+    </joint>
     <gazebo reference="lidar_frame_${lidar_prefix}">
       <material>Gazebo/Black</material>
       <sensor name="laser" type="gpu_lidar">
         <pose> 0 0 0 0 0 0 </pose>
-        <visualize>false</visualize>
+        <visualize>true</visualize>
         <update_rate>10</update_rate>
         <lidar>
@@ -78,6 +87,13 @@
         </lidar>
         <topic>scan</topic>
-        <gz_frame_id>lidar_frame_${lidar_prefix}</gz_frame_id>
+        <gz_frame_id>lidar_beam_${lidar_prefix}</gz_frame_id>
       </sensor>
+      <!-- Add the gazebo_ros plugin -->
+      <plugin name="gazebo_ros_laser_controller" filename="libgazebo_ros_gpu_laser.so">
+        <alwaysOn>true</alwaysOn>
+        <updateRate>10</updateRate>
+        <topicName>/scan</topicName>
+        <frameName>lidar_beam_${lidar_prefix}</frameName>
+      </plugin>
     </gazebo>
   </xacro:macro>

Commit message: harmonic fixes

File: description/urdf/ld06.urdf.xacro (robot description, xacro)
@@ -35,5 +35,5 @@
         <material name="ld06_${lidar_prefix}_grey" />
       </visual>
-      <visual> <!-- box-->
+      <visual>
         <origin xyz="0 0.017 ${ld06_base_box_height + (ld06_box_height / 2)}" rpy="0 0 0" />
         <geometry>
@@ -42,5 +42,5 @@
         <material name="ld06_${lidar_prefix}_blackish" />
       </visual>
-      <visual> <!-- cylinder -->
+      <visual>
         <origin
           xyz="0 0.017 ${(ld06_base_box_height + ld06_box_height) +(ld06_cylinder_height / 2)}"
@@ -51,5 +51,5 @@
         <material name="ld06_${lidar_prefix}_cylinder" />
       </visual>
-      <visual> <!-- base_cylinder -->
+      <visual>
         <geometry>
           <cylinder radius="${ld06_base_box_width / 2}" length="${ld06_base_box_height}" />
@@ -69,6 +69,5 @@
     <gazebo reference="lidar_frame_${lidar_prefix}">
       <material>Gazebo/Black</material>
-      <sensor name="laser" type="gpu_lidar">
-        <pose> 0 0 0 0 0 0 </pose>
+      <sensor name="lidar_frame_${lidar_prefix}" type="gpu_lidar">
         <visualize>true</visualize>
         <update_rate>10</update_rate>

Commit message: More gazebo tweaks

File: description/urdf/ld06.urdf.xacro (robot description, xacro)
@@ -43,7 +43,5 @@
       </visual>
       <visual>
-        <origin
-          xyz="0 0.017 ${(ld06_base_box_height + ld06_box_height) +(ld06_cylinder_height / 2)}"
-          rpy="0 0 0" />
+        <origin xyz="0 0.017 ${(ld06_base_box_height + ld06_box_height) +(ld06_cylinder_height / 2)}" rpy="0 0 0" />
         <geometry>
           <cylinder radius="${ld06_cylinder_radius}" length="${ld06_cylinder_height}" />
@@ -58,6 +56,5 @@
         <origin xyz="0 ${ld06_base_box_width / 4} ${(ld06_base_box_height / 2)}" rpy="0 0 0" />
       </visual>
-      <xacro:solid_cuboid_inertial rpy="0 0 0" xyz="0 0 0" mass_kg="0.001"
-        x="${ld06_base_box_width}" y="${ld06_base_box_width / 2}" z="${ld06_base_box_height}" />
+      <xacro:solid_cuboid_inertial rpy="0 0 0" xyz="0 0 0" mass_kg="0.001" x="${ld06_base_box_width}" y="${ld06_base_box_width / 2}" z="${ld06_base_box_height}" />
     </link>
     <link name="lidar_beam_${lidar_prefix}"></link>
@@ -76,11 +73,18 @@
             <horizontal>
               <samples>450</samples>
+              <resolution>1</resolution>
               <min_angle>-3.14</min_angle>
               <max_angle>3.14</max_angle>
             </horizontal>
+            <vertical>
+              <samples>1</samples>
+              <resolution>1</resolution>
+              <min_angle>0</min_angle>
+              <max_angle>0</max_angle>
+            </vertical>
           </scan>
           <range>
             <min>0.3</min>
-            <max>12</max>
+            <max>12.0</max>
           </range>
         </lidar>

File: description/urdf/sigyn.urdf.xacro (robot description, xacro)
@@ -1,4 +1,7 @@
 <?xml version="1.0"?>
 <robot xmlns:xacro="http://ros.org/wiki/xacro" name="Sigyn">
+  <self_collide>false</self_collide>
+  <pose>0 0 0.2 0 0 0</pose>
+  <static>false</static>
   <xacro:arg name="use_ros2_control" default="true" />
   <xacro:arg name="sim_mode" default="false" />

Commit message: Saving stuff that will probably be archived soon.

File: description/urdf/ld06.urdf.xacro (robot description, xacro)
@@ -24,4 +24,5 @@
     <link name="lidar_frame_${lidar_prefix}">
       <collision>
+        <origin xyz="0 0 ${ld06_base_box_height / 2}" rpy="0 0 0" />
         <geometry>
           <box size="${ld06_base_box_width} ${ld06_base_box_width / 2} ${ld06_base_box_height}" />
@@ -74,6 +75,6 @@
               <samples>450</samples>
               <resolution>1</resolution>
-              <min_angle>-3.14</min_angle>
-              <max_angle>3.14</max_angle>
+              <min_angle>-3.14159</min_angle>
+              <max_angle>3.14159</max_angle>
             </horizontal>
             <vertical>
@@ -88,14 +89,36 @@
             <max>12.0</max>
           </range>
+          <noise>
+            <type>gaussian</type>
+            <mean>0.0</mean>
+            <stddev>0.01</stddev>
+          </noise>
+          <!-- Add ray filtering to handle self-collisions -->
+          <ray>
+            <scan>
+              <horizontal>
+                <samples>450</samples>
+                <resolution>1</resolution>
+                <min_angle>-3.14159</min_angle>
+                <max_angle>3.14159</max_angle>
+              </horizontal>
+            </scan>
+            <range>
+              <min>0.3</min>
+              <max>12.0</max>
+            </range>
+          </ray>
         </lidar>
         <topic>scan</topic>
         <gz_frame_id>lidar_beam_${lidar_prefix}</gz_frame_id>
       </sensor>
-      <!-- Add the gazebo_ros plugin -->
+      <!-- Use correct Gazebo Garden/Harmonic plugin -->
       <plugin name="gazebo_ros_laser_controller" filename="libgazebo_ros_gpu_laser.so">
-        <alwaysOn>true</alwaysOn>
-        <updateRate>10</updateRate>
-        <topicName>/scan</topicName>
-        <frameName>lidar_beam_${lidar_prefix}</frameName>
+        <ros>
+          <namespace></namespace>
+          <remapping>~/out:=scan</remapping>
+        </ros>
+        <output_type>sensor_msgs/LaserScan</output_type>
+        <frame_name>lidar_beam_${lidar_prefix}</frame_name>
       </plugin>
     </gazebo>

Commit message: Snapshot and also recovering lost files

File: description/urdf/ld06.urdf.xacro (robot description, xacro)
@@ -60,5 +60,5 @@
     </link>
     <link name="lidar_beam_${lidar_prefix}"></link>
-    <joint name="laser_beam_joint" type="fixed">
+    <joint name="laser_beam_${lidar_prefix}_joint" type="fixed">
       <parent link="lidar_frame_${lidar_prefix}" />
       <child link="lidar_beam_${lidar_prefix}" />
@@ -125,5 +125,5 @@
   </xacro:macro>
   <!--
-Copyright (c) 2024 Michael Wimble
+Copyright (c) 2025 Michael Wimble
 Permission is hereby granted, free of charge, to any person obtaining a copy
 of this software and associated documentation files (the "Software"), to deal

File: description/urdf/sigyn.urdf.xacro (robot description, xacro)
@@ -23,8 +23,11 @@
   <xacro:caster_wheel config="${props}" />
   <xacro:include filename="$(find description)/urdf/ld06.urdf.xacro" />
-  <xacro:include filename="$(find description)/urdf/gazebo.urdf.xacro" />
   <xacro:ld06 lidar_prefix="top_lidar">
     <origin xyz="0.155 0 0.300" rpy="0 0 -${pi / 2}" />
   </xacro:ld06>
+  <xacro:ld06 lidar_prefix="cup_lidar">
+    <origin xyz="${0.155-0.34} 0 ${0.300+1.485}" rpy="0 0 0" />
+  </xacro:ld06>
+  <xacro:include filename="$(find description)/urdf/gazebo.urdf.xacro" />
   <xacro:include filename="$(find description)/urdf/gripper_assembly.urdf.xacro" />
   <joint name="base_link_to_elevator_pole" type="fixed">
@@ -111,3 +114,4 @@
   </joint>
   <link name="imu_1" />
+  <xacro:include filename="$(find description)/urdf/vl53l0x.xacro" />
 </robot>

Commit message: Fixes for simulation

File: description/urdf/ld06.urdf.xacro (robot description, xacro)
@@ -1,5 +1,5 @@
 <?xml version="1.0"?>
 <robot xmlns:xacro="http://ros.org/wiki/xacro" name="ld06">
-  <xacro:macro name="ld06" params="lidar_prefix *joint_pose">
+  <xacro:macro name="ld06" params="lidar_prefix topic_name:=scan *joint_pose">
     <material name="ld06_${lidar_prefix}_grey">
       <color rgba="0.3 0.3 0.3 1" />
@@ -110,5 +110,5 @@
           </ray>
         </lidar>
-        <topic>scan</topic>
+        <topic>${topic_name}</topic>
         <gz_frame_id>lidar_beam_${lidar_prefix}</gz_frame_id>
       </sensor>
@@ -117,5 +117,5 @@
         <ros>
           <namespace></namespace>
-          <remapping>~/out:=scan</remapping>
+          <remapping>~/out:=${topic_name}</remapping>
         </ros>
         <output_type>sensor_msgs/LaserScan</output_type>

File: description/urdf/oakd.urdf.xacro (robot description, xacro)
@@ -27,5 +27,5 @@
         <origin rpy="0 0 0" xyz="0 0 0" />
         <geometry>
-          <mesh filename="package://depthai_descriptions/urdf/models/OAK-D-PRO.stl" />
+          <mesh filename="package://description/meshes/OAK-D.dae" />
         </geometry>
         <material name="mat">

File: description/urdf/sigyn.urdf.xacro (robot description, xacro)
@@ -9,5 +9,10 @@
   <xacro:include filename="$(find description)/urdf/sigyn_caster_wheel_macro.urdf.xacro" />
   <xacro:include filename="$(find description)/urdf/sigyn_wheels_macro.urdf.xacro" />
-  <xacro:include filename="$(find description)/urdf/oakd.urdf.xacro" />
+  <xacro:unless value="$(arg sim_mode)">
+    <xacro:include filename="$(find description)/urdf/depthai_macro.urdf.xacro" />
+  </xacro:unless>
+  <xacro:unless value="$(arg sim_mode)">
+    <xacro:include filename="$(find description)/urdf/oakd.urdf.xacro" />
+  </xacro:unless>
   <xacro:if value="$(arg use_ros2_control)">
     <xacro:include filename="ros2_control.xacro" />
@@ -23,8 +28,8 @@
   <xacro:caster_wheel config="${props}" />
   <xacro:include filename="$(find description)/urdf/ld06.urdf.xacro" />
-  <xacro:ld06 lidar_prefix="top_lidar">
+  <xacro:ld06 lidar_prefix="top_lidar" topic_name="scan">
     <origin xyz="0.155 0 0.300" rpy="0 0 -${pi / 2}" />
   </xacro:ld06>
-  <xacro:ld06 lidar_prefix="cup_lidar">
+  <xacro:ld06 lidar_prefix="cup_lidar" topic_name="scan_cup">
     <origin xyz="${0.155-0.34} 0 ${0.300+1.485}" rpy="0 0 0" />
   </xacro:ld06>
@@ -37,9 +42,12 @@
   </joint>
   <!-- <xacro:oakd_link mount_point="elevator_top" /> -->
-  <xacro:oakd_joint mount_point="elevator_top">
-    <origin xyz="-0.12 -0.02 1.47" rpy="0 ${(pi / 4)+13*(2.0*pi/360.0)} ${-0*(2.0*pi/360.0)}" />
-  </xacro:oakd_joint>
+  <xacro:unless value="$(arg sim_mode)">
+    <xacro:oakd_joint mount_point="elevator_top">
+      <origin xyz="-0.12 -0.02 1.47" rpy="0 ${(pi / 4)+13*(2.0*pi/360.0)} ${-0*(2.0*pi/360.0)}" />
+    </xacro:oakd_joint>
+  </xacro:unless>
   <gazebo>
-    <plugin filename="gz-sim-joint-position-controller-system" name="gz::sim::systems::JointPositionController">
+    <plugin filename="gz-sim-joint-position-controller-system"
+      name="gz::sim::systems::JointPositionController">
       <joint_name>elevator_pole_to_elevator_connector_plate</joint_name>
       <p_gain>1.0</p_gain>
@@ -52,5 +60,6 @@
       <topic>/elevator_connector_plate/position</topic>
     </plugin>
-    <plugin filename="gz-sim-joint-position-controller-system" name="gz::sim::systems::JointPositionController">
+    <plugin filename="gz-sim-joint-position-controller-system"
+      name="gz::sim::systems::JointPositionController">
       <joint_name>gripper_elevator_plate_to_gripper_extender</joint_name>
       <p_gain>1.0</p_gain>
@@ -63,5 +72,6 @@
       <topic>/gripper_elevator_plate_to_gripper_extender/position</topic>
     </plugin>
-    <plugin filename="gz-sim-joint-position-controller-system" name="gz::sim::systems::JointPositionController">
+    <plugin filename="gz-sim-joint-position-controller-system"
+      name="gz::sim::systems::JointPositionController">
       <joint_name>gripper_wrist_to_parallel_gripper_base_plate</joint_name>
       <p_gain>1.0</p_gain>
@@ -74,5 +84,6 @@
       <topic>/gripper_wrist_to_parallel_gripper_base_plate/position</topic>
     </plugin>
-    <plugin filename="gz-sim-joint-position-controller-system" name="gz::sim::systems::JointPositionController">
+    <plugin filename="gz-sim-joint-position-controller-system"
+      name="gz::sim::systems::JointPositionController">
       <joint_name>parallel_gripper_base_plate_to_left_finger</joint_name>
       <p_gain>1.0</p_gain>
@@ -85,5 +96,6 @@
       <topic>/parallel_gripper_base_plate_to_left_finger/position</topic>
     </plugin>
-    <plugin filename="gz-sim-joint-position-controller-system" name="gz::sim::systems::JointPositionController">
+    <plugin filename="gz-sim-joint-position-controller-system"
+      name="gz::sim::systems::JointPositionController">
       <joint_name>parallel_gripper_base_plate_to_right_finger</joint_name>
       <p_gain>1.0</p_gain>
@@ -97,5 +109,6 @@
     </plugin>
   </gazebo>
-  <xacro:diff_drive_controller config="${props}" instances1="${props.wheels.instances}" instances2="${props.wheels.instances}" />
+  <xacro:diff_drive_controller config="${props}" instances1="${props.wheels.instances}"
+    instances2="${props.wheels.instances}" />
   <!-- IMU0 - Upside down & backwards -->
   <joint name="imu0_joint" type="fixed">
