Commit message: Tilt up the VL53L0X by half the field of view

File: description/urdf/vl53l0x.xacro (robot description, xacro)
@@ -37,5 +37,5 @@
     <child link="vl53l0x_0" />
     <parent link="base_link" />
-    <origin xyz="-0.165 -0.150 0.050" rpy="${pi/2.0} 0 -${pi}" />
+    <origin xyz="-0.165 -0.150 0.050" rpy="${pi/2.0} -0.218 -${pi}" />
   </joint>
   <link name="vl53l0x_1">
@@ -51,5 +51,5 @@
     <child link="vl53l0x_1" />
     <parent link="base_link" />
-    <origin xyz="-0.145 -0.165 0.050" rpy="${pi/2.0} 0 -${pi/2.0}" />
+    <origin xyz="-0.145 -0.165 0.050" rpy="${pi/2.0} -0.218 -${pi/2.0}" />
   </joint>
   <link name="vl53l0x_2">
@@ -65,5 +65,5 @@
     <child link="vl53l0x_2" />
     <parent link="base_link" />
-    <origin xyz="0.145 -0.165 0.050" rpy="${pi/2.0} 0 -${pi/2.0}" />
+    <origin xyz="0.145 -0.165 0.050" rpy="${pi/2.0} -0.218 -${pi/2.0}" />
   </joint>
   <link name="vl53l0x_3">
@@ -79,5 +79,5 @@
     <child link="vl53l0x_3" />
     <parent link="base_link" />
-    <origin xyz="0.160 -0.150 0.050" rpy="${pi/2.0} 0 0" />
+    <origin xyz="0.160 -0.150 0.050" rpy="${pi/2.0} -0.218 0" />
   </joint>
   <link name="vl53l0x_4">
@@ -93,5 +93,5 @@
     <child link="vl53l0x_4" />
     <parent link="base_link" />
-    <origin xyz="0.160 0.150 0.050" rpy="${pi/2.0} 0 0" />
+    <origin xyz="0.160 0.150 0.050" rpy="${pi/2.0} -0.218 0" />
   </joint>
   <link name="vl53l0x_5">
@@ -107,5 +107,5 @@
     <child link="vl53l0x_5" />
     <parent link="base_link" />
-    <origin xyz="0.145 0.165 0.200" rpy="${pi/2.0} 0 ${pi/2.0}" />
+    <origin xyz="0.145 0.165 0.200" rpy="${pi/2.0} -0.218 ${pi/2.0}" />
   </joint>
   <link name="vl53l0x_6">
@@ -121,5 +121,5 @@
     <child link="vl53l0x_6" />
     <parent link="base_link" />
-    <origin xyz="-0.145 0.165 0.050" rpy="${pi/2.0} 0 ${pi/2.0}" />
+    <origin xyz="-0.145 0.165 0.050" rpy="${pi/2.0} -0.218 ${pi/2.0}" />
   </joint>
     <link name="vl53l0x_7">
@@ -135,5 +135,5 @@
     <child link="vl53l0x_7" />
     <parent link="base_link" />
-    <origin xyz="-0.165 0.150 0.050" rpy="${pi/2.0} 0 -${pi}" />
+    <origin xyz="-0.165 0.150 0.050" rpy="${pi/2.0} -0.218 -${pi}" />
   </joint>
 </robot>
