Commit message: Added OAK-D pointcloud. Removed unused stuff.

File: description/urdf/oakd.urdf.xacro (robot description, xacro)
@@ -6,74 +6,79 @@
 <!--  xacro macros for oakd mount -->
 <robot name="oakd" xmlns:xacro="http://ros.org/wiki/xacro">
-  <xacro:macro name="oakd_link" params="mount_point">
-    <xacro:property name="oakd_length" value="0.0803" />
-    <xacro:property name="oakd_width" value="0.0957" />
-    <xacro:property name="oakd_depth" value="0.1267" />
-    <xacro:property name="oakd_mass" value="0.15" />
-    <link name="oakd_${mount_point}">
-      <pose>0.0 0.0 0.0 0.0 0.0 0.0</pose>
+  <xacro:macro name="oakd_joint" params="mount_point *joint_pose">
+    <joint name="oakd_joint_${mount_point}" type="fixed">
+      <parent link="base_link" />
+      <child link="oak-d-base-frame" />
+      <xacro:insert_block name="joint_pose" />
+    </joint>
+    <!--
+    <gazebo reference="oakd_joint_${mount_point}">
+      <preserveFixedJoint>true</preserveFixedJoint>
+    </gazebo> -->
+    <link name="oak-d-base-frame" /> <!-- base_link of the sensor-->
+    <link name="oak" />
+    <joint name="oak_center_joint" type="fixed">
+      <parent link="oak-d-base-frame" />
+      <child link="oak" />
+      <origin rpy="0.0 0.0 0.0" xyz="0.0 0.0 0.0" />
+    </joint>
+    <link name="oak_model_origin">
       <visual>
         <origin rpy="0 0 0" xyz="0 0 0" />
         <geometry>
-          <!-- <box size="${oakd_length} ${oakd_width} ${oakd_depth}" /> -->
-          <mesh filename="file://$(find description)/meshes/OAK-D.dae" />
+          <mesh filename="package://depthai_descriptions/urdf/models/OAK-D-PRO.stl" />
         </geometry>
-        <color rgba="0.15 0.15 0.15 1" />
+        <material name="mat">
+          <color rgba="0.8 0.8 0.8 0.8" />
+        </material>
       </visual>
-      <collision>
-        <origin rpy="0 0 0" xyz="0 0 0" />
-        <geometry>
-          <box size="${oakd_length} ${oakd_width} ${oakd_depth}" />
-        </geometry>
-      </collision>
-      <xacro:solid_cuboid_inertial
-        rpy="0 0 0" xyz="0 0 0"
-        mass_kg="${oakd_mass}"
-        x="${oakd_length}" y="${oakd_width}" z="${oakd_depth}" />
     </link>
-    <gazebo reference="oakd_${mount_point}">
-      <material>Gazebo/Red</material>
-      <sensor name="camera_${mount_point}" type="camera">
-        <always_on>true</always_on>
-        <visualize>true</visualize>
-        <update_rate>10</update_rate>
-        <camera name='__default__'>
-          <horizontal_fov>1.089</horizontal_fov>
-          <image>
-            <format>R8G8B8</format>
-            <width>640</width>
-            <height>480</height>
-          </image>
-          <clip>
-            <near>0.05</near>
-            <far>8.0</far>
-          </clip>
-        </camera>
-        <plugin name='camera_controller_${mount_point}' filename='libgazebo_ros_camera.so'>
-          <alwaysOn>1</alwaysOn>
-          <updateRate>0.0</updateRate>
-          <cameraName>camera_${mount_point}</cameraName>
-          <hackBaseline>0.07</hackBaseline>
-          <distortionK1>0.0</distortionK1>
-          <distortionK2>0.0</distortionK2>
-          <distortionK3>0.0</distortionK3>
-          <distortionT1>0.0</distortionT1>
-          <distortionT2>0.0</distortionT2>
-        </plugin>
-      </sensor>
-    </gazebo>
-    <gazebo reference="oakd_joint_${mount_point}">
-    </gazebo>
-  </xacro:macro>
-  <xacro:macro name="oakd_joint" params="mount_point *joint_pose">
-    <joint name="oakd_joint_${mount_point}" type="fixed">
-      <!-- <origin rpy="${roll} ${pitch} ${yaw}" xyz="${x}+0.1 ${y}-0.01 ${z}" /> -->
-      <parent link="base_link" />
-      <child link="oakd_${mount_point}" />
-      <xacro:insert_block name="joint_pose" />
+    <joint name="oak_model_origin_joint" type="fixed">
+      <parent link="oak" />
+      <child link="oak_model_origin" />
+      <origin rpy="1.5708 0 1.5708" xyz="0 0 0" />
+    </joint> <!-- IMU -->
+    <link name="oak_imu_frame" />
+    <joint name="oak_imu_joint" type="fixed">
+      <parent link="oak" />
+      <child link="oak_imu_frame" />
+      <origin rpy="3.141592653589793 1.5707963267948966 0.0" xyz="-0.008 -0.037945 -0.00079" />
     </joint>
-    <gazebo reference="oakd_joint_${mount_point}">
-      <preserveFixedJoint>true</preserveFixedJoint>
-    </gazebo>
+    <link name="oak_rgb_camera_frame" />
+    <joint name="oak_rgb_camera_joint" type="fixed">
+      <parent link="oak" />
+      <child link="oak_rgb_camera_frame" />
+      <origin rpy="0 0 0" xyz="0 0 0" />
+    </joint>
+    <link name="oak_rgb_camera_optical_frame" />
+    <joint name="oak_rgb_camera_optical_joint" type="fixed">
+      <origin rpy="-1.5707963267948966 0.0 -1.5707963267948966" xyz="0 0 0" />
+      <parent link="oak_rgb_camera_frame" />
+      <child link="oak_rgb_camera_optical_frame" />
+    </joint> <!-- Left Camera -->
+    <link name="oak_left_camera_frame" />
+    <joint name="oak_left_camera_joint" type="fixed">
+      <parent link="oak" />
+      <child link="oak_left_camera_frame" />
+      <origin rpy="0 0 0" xyz="0 0.0375 0" />
+    </joint>
+    <link name="oak_left_camera_optical_frame" />
+    <joint name="oak_left_camera_optical_joint" type="fixed">
+      <origin rpy="-1.5707963267948966 0.0 -1.5707963267948966" xyz="0 0 0" />
+      <parent link="oak_left_camera_frame" />
+      <child link="oak_left_camera_optical_frame" />
+    </joint> <!-- right Camera -->
+    <link name="oak_right_camera_frame" />
+    <joint name="oak_right_camera_joint" type="fixed">
+      <parent link="oak" />
+      <child link="oak_right_camera_frame" />
+      <origin rpy="0 0 0" xyz="0 -0.0375 0" />
+    </joint>
+    <link name="oak_right_camera_optical_frame" />
+    <joint name="oak_right_camera_optical_joint" type="fixed">
+      <origin rpy="-1.5707963267948966 0.0 -1.5707963267948966" xyz="0 0 0" />
+      <parent link="oak_right_camera_frame" />
+      <child link="oak_right_camera_optical_frame" />
+    </joint>
   </xacro:macro>
 </robot>

File: description/urdf/sigyn.urdf.xacro (robot description, xacro)
@@ -12,4 +12,5 @@
   <xacro:include filename="$(find description)/urdf/sigyn_caster_wheel_macro.urdf.xacro" />
   <xacro:include filename="$(find description)/urdf/sigyn_wheels_macro.urdf.xacro" />
+  <xacro:include filename="$(find description)/urdf/oakd.urdf.xacro" />
   <xacro:if value="$(arg use_ros2_control)">
     <xacro:include filename="ros2_control.xacro" />
@@ -31,10 +32,15 @@
   <xacro:include filename="$(find description)/urdf/gripper_assembly.urdf.xacro" />
   <joint name="base_link_to_elevator_pole" type="fixed">
-    <origin xyz="-0.16 0.015 ${0.3 + (elevator_pole_height/2)}" rpy="0 0 0" />
+    <origin xyz="-0.16 -0.015 ${0.3 + (elevator_pole_height/2)}" rpy="0 0 0" />
     <parent link="base_link" />
     <child link="evelator_pole" />
   </joint>
+  <!-- <xacro:oakd_link mount_point="elevator_top" /> -->
+  <xacro:oakd_joint mount_point="elevator_top">
+    <origin xyz="-0.12 -0.02 1.5" rpy="0 ${(pi / 4)+9*(2.0*pi/360.0)} ${-9*(2.0*pi/360.0)}" />
+  </xacro:oakd_joint>
   <gazebo>
-    <plugin filename="gz-sim-joint-position-controller-system" name="gz::sim::systems::JointPositionController">
+    <plugin filename="gz-sim-joint-position-controller-system"
+      name="gz::sim::systems::JointPositionController">
       <joint_name>elevator_pole_to_elevator_connector_plate</joint_name>
       <p_gain>1.0</p_gain>
@@ -47,5 +53,6 @@
       <topic>/elevator_connector_plate/position</topic>
     </plugin>
-    <plugin filename="gz-sim-joint-position-controller-system" name="gz::sim::systems::JointPositionController">
+    <plugin filename="gz-sim-joint-position-controller-system"
+      name="gz::sim::systems::JointPositionController">
       <joint_name>gripper_elevator_plate_to_gripper_extender</joint_name>
       <p_gain>1.0</p_gain>
@@ -58,5 +65,6 @@
       <topic>/gripper_elevator_plate_to_gripper_extender/position</topic>
     </plugin>
-    <plugin filename="gz-sim-joint-position-controller-system" name="gz::sim::systems::JointPositionController">
+    <plugin filename="gz-sim-joint-position-controller-system"
+      name="gz::sim::systems::JointPositionController">
       <joint_name>gripper_wrist_to_parallel_gripper_base_plate</joint_name>
       <p_gain>1.0</p_gain>
@@ -69,5 +77,6 @@
       <topic>/gripper_wrist_to_parallel_gripper_base_plate/position</topic>
     </plugin>
-    <plugin filename="gz-sim-joint-position-controller-system" name="gz::sim::systems::JointPositionController">
+    <plugin filename="gz-sim-joint-position-controller-system"
+      name="gz::sim::systems::JointPositionController">
       <joint_name>parallel_gripper_base_plate_to_left_finger</joint_name>
       <p_gain>1.0</p_gain>
@@ -80,5 +89,6 @@
       <topic>/parallel_gripper_base_plate_to_left_finger/position</topic>
     </plugin>
-    <plugin filename="gz-sim-joint-position-controller-system" name="gz::sim::systems::JointPositionController">
+    <plugin filename="gz-sim-joint-position-controller-system"
+      name="gz::sim::systems::JointPositionController">
       <joint_name>parallel_gripper_base_plate_to_right_finger</joint_name>
       <p_gain>1.0</p_gain>
@@ -92,4 +102,5 @@
     </plugin>
   </gazebo>
-  <xacro:diff_drive_controller config="${props}" instances1="${props.wheels.instances}" instances2="${props.wheels.instances}" />
+  <xacro:diff_drive_controller config="${props}" instances1="${props.wheels.instances}"
+    instances2="${props.wheels.instances}" />
 </robot>

Commit message: snapshot

File: description/urdf/oakd.urdf.xacro (robot description, xacro)
@@ -6,4 +6,6 @@
 <!--  xacro macros for oakd mount -->
 <robot name="oakd" xmlns:xacro="http://ros.org/wiki/xacro">
+  <!-- Resolve package share to absolute path so Gazebo can load meshes reliably -->
+  <xacro:property name="description_share" value="$(find description)"/>
   <xacro:macro name="oakd_joint" params="mount_point *joint_pose">
     <joint name="oakd_joint_${mount_point}" type="fixed">
@@ -27,5 +29,6 @@
         <origin rpy="0 0 0" xyz="0 0 0" />
         <geometry>
-          <mesh filename="package://description/meshes/OAK-D.dae" />
+          <!-- Use absolute file URI to avoid model:// resolution issues in Gazebo -->
+          <mesh filename="file://${description_share}/meshes/OAK-D.dae" scale="0.001 0.001 0.001" />
         </geometry>
         <material name="mat">
@@ -33,4 +36,15 @@
         </material>
       </visual>
+      <collision>
+        <origin rpy="0 0 0" xyz="0 0 0" />
+        <geometry>
+          <box size="0.098 0.030 0.025" />
+        </geometry>
+      </collision>
+      <inertial>
+        <mass value="0.065" />
+        <origin xyz="0 0 0" rpy="0 0 0" />
+        <inertia ixx="0.0001" ixy="0" ixz="0" iyy="0.0001" iyz="0" izz="0.0001" />
+      </inertial>
     </link>
     <joint name="oak_model_origin_joint" type="fixed">
@@ -51,5 +65,5 @@
       <origin rpy="0 0 0" xyz="0 0 0" />
     </joint>
-    <link name="oak_rgb_camera_optical_frame" />
+  <!-- link defined with inertial below -->
     <joint name="oak_rgb_camera_optical_joint" type="fixed">
       <origin rpy="-1.5707963267948966 0.0 -1.5707963267948966" xyz="0 0 0" />
@@ -57,4 +71,16 @@
       <child link="oak_rgb_camera_optical_frame" />
     </joint> <!-- Left Camera -->
+    <!-- Minimal inertial to keep optical frame modeled in SDF -->
+    <link name="oak_rgb_camera_optical_frame">
+      <inertial>
+        <mass value="1e-6" />
+        <origin xyz="0 0 0" rpy="0 0 0" />
+        <inertia ixx="1e-9" ixy="0" ixz="0" iyy="1e-9" iyz="0" izz="1e-9" />
+      </inertial>
+    </link>
+    <!-- Preserve optical joint to avoid link lumping in Gazebo -->
+    <gazebo reference="oak_rgb_camera_optical_joint">
+      <preserveFixedJoint>true</preserveFixedJoint>
+    </gazebo>
     <link name="oak_left_camera_frame" />
     <joint name="oak_left_camera_joint" type="fixed">
@@ -63,5 +89,5 @@
       <origin rpy="0 0 0" xyz="0 0.0375 0" />
     </joint>
-    <link name="oak_left_camera_optical_frame" />
+  <!-- link defined with inertial below -->
     <joint name="oak_left_camera_optical_joint" type="fixed">
       <origin rpy="-1.5707963267948966 0.0 -1.5707963267948966" xyz="0 0 0" />
@@ -69,4 +95,16 @@
       <child link="oak_left_camera_optical_frame" />
     </joint> <!-- right Camera -->
+    <!-- Minimal inertial to keep optical frame modeled in SDF -->
+    <link name="oak_left_camera_optical_frame">
+      <inertial>
+        <mass value="1e-6" />
+        <origin xyz="0 0 0" rpy="0 0 0" />
+        <inertia ixx="1e-9" ixy="0" ixz="0" iyy="1e-9" iyz="0" izz="1e-9" />
+      </inertial>
+    </link>
+    <!-- Preserve optical joint to avoid link lumping in Gazebo -->
+    <gazebo reference="oak_left_camera_optical_joint">
+      <preserveFixedJoint>true</preserveFixedJoint>
+    </gazebo>
     <link name="oak_right_camera_frame" />
     <joint name="oak_right_camera_joint" type="fixed">
@@ -75,5 +113,12 @@
       <origin rpy="0 0 0" xyz="0 -0.0375 0" />
     </joint>
-    <link name="oak_right_camera_optical_frame" />
+    <link name="oak_right_camera_optical_frame">
+      <!-- Optional inertial to future-proof if attaching sensors later -->
+      <inertial>
+        <mass value="1e-6" />
+        <origin xyz="0 0 0" rpy="0 0 0" />
+        <inertia ixx="1e-9" ixy="0" ixz="0" iyy="1e-9" iyz="0" izz="1e-9" />
+      </inertial>
+    </link>
     <joint name="oak_right_camera_optical_joint" type="fixed">
       <origin rpy="-1.5707963267948966 0.0 -1.5707963267948966" xyz="0 0 0" />
@@ -81,4 +126,76 @@
       <child link="oak_right_camera_optical_frame" />
     </joint>
+        <!-- Gazebo-specific elements -->
+    <gazebo reference="oak_model_origin">
+      <material>Gazebo/DarkGrey</material>
+    </gazebo>
+    <!-- Attach sensors directly to optical frames with identity pose -->
+    <gazebo reference="oak_rgb_camera_optical_frame">
+      <sensor name="rgb_camera" type="camera">
+        <!-- Nudge sensor a bit forward along optical Z so it sees past the mount -->
+        <pose>0 0 0.05 0 0 0</pose>
+        <camera>
+          <horizontal_fov>1.089</horizontal_fov>
+          <image>
+            <width>640</width>
+            <height>480</height>
+            <format>R8G8B8</format>
+          </image>
+          <clip>
+            <near>0.1</near>
+            <far>100.0</far>
+          </clip>
+          <noise>
+            <type>gaussian</type>
+            <mean>0</mean>
+            <stddev>0.007</stddev>
+          </noise>
+        </camera>
+        <always_on>1</always_on>
+        <update_rate>30</update_rate>
+        <visualize>true</visualize>
+        <!-- Standard camera topic convention: base/image_raw and base/camera_info -->
+        <topic>oakd_top/color/image_raw</topic>
+        <!-- Ensure ROS frame_id is correct on the bridge -->
+        <gz_frame_id>oak_rgb_camera_optical_frame</gz_frame_id>
+      </sensor>
+    </gazebo>
+    <gazebo reference="oak_left_camera_optical_frame">
+      <!-- Depth + Point Cloud using single rgbd_camera sensor -->
+      <!-- rgbd_camera publishes: base/image, base/depth_image, base/points, base/camera_info -->
+      <sensor name="stereo_camera" type="rgbd_camera">
+        <!-- Nudge sensor forward to avoid self-occlusion by the mount -->
+        <pose>0 0 0.05 0 0 0</pose>
+        <camera>
+          <horizontal_fov>1.089</horizontal_fov>
+          <image>
+            <width>640</width>
+            <height>480</height>
+            <format>R8G8B8</format>
+          </image>
+          <depth_camera>
+            <clip>
+              <near>0.3</near>
+              <far>10.0</far>
+            </clip>
+          </depth_camera>
+          <clip>
+            <near>0.3</near>
+            <far>10.0</far>
+          </clip>
+          <noise>
+            <type>gaussian</type>
+            <mean>0</mean>
+            <stddev>0.1</stddev>
+          </noise>
+        </camera>
+        <always_on>1</always_on>
+        <update_rate>30</update_rate>
+        <visualize>false</visualize>
+        <!-- Base topic; Gazebo will append /image, /depth_image, /points, /camera_info -->
+        <topic>oakd_top/stereo</topic>
+        <gz_frame_id>oak_left_camera_optical_frame</gz_frame_id>
+      </sensor>
+    </gazebo>
   </xacro:macro>
 </robot>

File: description/urdf/sigyn.urdf.xacro (robot description, xacro)
@@ -12,7 +12,10 @@
     <xacro:include filename="$(find description)/urdf/depthai_macro.urdf.xacro" />
   </xacro:unless>
-  <xacro:unless value="$(arg sim_mode)">
+  <!-- <xacro:unless value="$(arg sim_mode)"> -->
     <xacro:include filename="$(find description)/urdf/oakd.urdf.xacro" />
-  </xacro:unless>
+  <!-- </xacro:unless> -->
+  <!-- <xacro:if value="$(arg sim_mode)">
+    <xacro:include filename="$(find description)/urdf/oakd_sim.urdf.xacro" />
+  </xacro:if> -->
   <xacro:if value="$(arg use_ros2_control)">
     <xacro:include filename="ros2_control.xacro" />
@@ -32,19 +35,21 @@
   </xacro:ld06>
   <xacro:ld06 lidar_prefix="cup_lidar" topic_name="scan_cup">
-    <origin xyz="${0.155-0.34} 0 ${0.300+1.485}" rpy="0 0 0" />
+    <!-- <origin xyz="${0.15-0.34} 0 ${0.300+1.485}" rpy="0 0 0" /> -->
+    <origin xyz="-0.161 -0.015 ${0.300 + 1.485 - 0.032}" rpy="0 0 0" />
   </xacro:ld06>
   <xacro:include filename="$(find description)/urdf/gazebo.urdf.xacro" />
   <xacro:include filename="$(find description)/urdf/gripper_assembly.urdf.xacro" />
   <joint name="base_link_to_elevator_pole" type="fixed">
-    <origin xyz="-0.16 -0.015 ${0.3 + (elevator_pole_height/2)}" rpy="0 0 0" />
+    <origin xyz="-0.16 0 ${0.3 + (elevator_pole_height/2)}" rpy="0 0 0" />
     <parent link="base_link" />
     <child link="evelator_pole" />
   </joint>
   <!-- <xacro:oakd_link mount_point="elevator_top" /> -->
-  <xacro:unless value="$(arg sim_mode)">
-    <xacro:oakd_joint mount_point="elevator_top">
-      <origin xyz="-0.12 -0.02 1.47" rpy="0 ${(pi / 4)+13*(2.0*pi/360.0)} ${-0*(2.0*pi/360.0)}" />
-    </xacro:oakd_joint>
-  </xacro:unless>
+  <xacro:oakd_joint mount_point="elevator_top">
+    <!-- <origin xyz="-0.12 -0.02 1.47" rpy="0 ${(pi / 4)+13*(2.0*pi/360.0)} ${-0*(2.0*pi/360.0)}" /> -->
+    <!-- <origin xyz="-0.12 -0.02 1.7" rpy="0 ${pi / 4} -1.029" /> -->
+    <!-- <origin xyz="-0.09 0.015 1.65" rpy="${-pi / 2} ${(-pi / 2) + 1.029} 0" /> -->
+    <origin xyz="-0.09 0.0 1.65" rpy="${-pi / 2} ${(-pi / 2) + 1.029} 0" />
+  </xacro:oakd_joint>
   <gazebo>
     <plugin filename="gz-sim-joint-position-controller-system"
