Commit message: Cameras now simulated

File: description/urdf/sim_cameras.urdf.xacro (robot description, xacro)
@@ -41,5 +41,5 @@
           </clip>
         </camera>
-        <topic>/oakd/image_raw</topic>
+        <topic>/oakd_top/color/image</topic>
         <gz_frame_id>oakd_sim_optical</gz_frame_id>
       </sensor>
@@ -51,5 +51,5 @@
       <parent link="${parent_link}"/>
       <child link="pi_camera_sim_link"/>
-      <origin xyz="0.05 0 0" rpy="0 0 0"/>
+      <origin xyz="0.0 0.1 -0.125" rpy="-${pi/2} -${pi/2} 0"/>
     </joint>
     <link name="pi_camera_sim_link">
@@ -86,5 +86,5 @@
           </clip>
         </camera>
-        <topic>/pi_camera/image_raw</topic>
+        <topic>/gripper/camera/image</topic>
         <gz_frame_id>pi_camera_sim_optical</gz_frame_id>
       </sensor>

Commit message: Snapshot

File: description/urdf/sim_cameras.urdf.xacro (robot description, xacro)
@@ -48,8 +48,12 @@
   <!-- Pi Camera for Simulation (on gripper for close-up centering) -->
   <xacro:macro name="pi_camera_sim" params="parent_link">
+    <!-- Pitch down angle in degrees -->
+    <xacro:property name="pitch_down_degrees" value="35"/>
     <joint name="pi_camera_sim_joint" type="fixed">
       <parent link="${parent_link}"/>
       <child link="pi_camera_sim_link"/>
-      <origin xyz="0.0 0.1 -0.125" rpy="-${pi/2} -${pi/2} 0"/>
+      <!-- Pitch calculation: -90 degrees (level) + pitch_down_degrees -->
+      <!-- Adjusted Y offset to 0.18 to ensure we peek OVER the gripper backplate. 35deg pitch. -->
+      <origin xyz="0.0 0.18 -0.125" rpy="0 -${(90 - pitch_down_degrees) * pi / 180.0} -${pi/2}"/>
     </joint>
     <link name="pi_camera_sim_link">

Commit message: Snapshot

File: description/urdf/sim_cameras.urdf.xacro (robot description, xacro)
@@ -55,5 +55,5 @@
       <!-- Pitch calculation: -90 degrees (level) + pitch_down_degrees -->
       <!-- Adjusted Y offset to 0.18 to ensure we peek OVER the gripper backplate. 35deg pitch. -->
-      <origin xyz="0.0 0.18 -0.125" rpy="0 -${(90 - pitch_down_degrees) * pi / 180.0} -${pi/2}"/>
+      <origin xyz="0.0 0.1 -0.06" rpy="0 -${(90 - pitch_down_degrees) * pi / 180.0} -${pi/2}"/>
     </joint>
     <link name="pi_camera_sim_link">

Commit message: Snapshot. Raises gripper to correct height to find can. Centers between gripper paddles.

File: description/urdf/sim_cameras.urdf.xacro (robot description, xacro)
@@ -49,5 +49,5 @@
   <xacro:macro name="pi_camera_sim" params="parent_link">
     <!-- Pitch down angle in degrees -->
-    <xacro:property name="pitch_down_degrees" value="35"/>
+    <xacro:property name="pitch_down_degrees" value="25"/>
     <joint name="pi_camera_sim_joint" type="fixed">
       <parent link="${parent_link}"/>
