Commit message: Snapshot, pi_servo working with parallel gripper

File: description/urdf/ros2_control.xacro (robot description, xacro)
@@ -9,5 +9,5 @@
         <param name="example_param_hw_slowdown">1.23</param>
       </hardware>
-      <joint name="servo1_joint">
+      <joint name="parallel_gripper_base_plate_to_left_finger">
         <command_interface name="position">
           <param name="min">-100</param>

Commit message: Start of ros2_control for the roboclaw.

File: description/urdf/ros2_control.xacro (robot description, xacro)
@@ -45,4 +45,33 @@
       </joint>
     </ros2_control> -->
+    <!-- Sigyn Differential Drive System -->
+    <ros2_control name="sigyn_system" type="system">
+      <hardware>
+        <plugin>sigyn_hardware_interface/SigynSystem</plugin>
+        <param name="port">/dev/teensy_sensor</param>
+        <param name="baud_rate">921600</param>
+        <param name="wheel_diameter">0.102224144529039</param>
+        <param name="wheel_base">0.3906</param>
+        <param name="pulses_per_revolution">1000</param>
+        <param name="command_timeout">0.5</param>
+        <param name="read_timeout">0.1</param>
+      </hardware>
+      <joint name="left_wheel_joint">
+        <command_interface name="velocity">
+          <param name="min">-10.0</param>
+          <param name="max">10.0</param>
+        </command_interface>
+        <state_interface name="position"/>
+        <state_interface name="velocity"/>
+      </joint>
+      <joint name="right_wheel_joint">
+        <command_interface name="velocity">
+          <param name="min">-10.0</param>
+          <param name="max">10.0</param>
+        </command_interface>
+        <state_interface name="position"/>
+        <state_interface name="velocity"/>
+      </joint>
+    </ros2_control>
   </xacro:unless>
   <xacro:if value="$(arg sim_mode)">

Commit message: Gripper working again

File: description/urdf/ros2_control.xacro (robot description, xacro)
@@ -105,5 +105,5 @@
         <state_interface name="position"/>
       </joint>
-      <joint name="parallel_gripper_base_plate_to_left_finger">
+      <!-- <joint name="parallel_gripper_base_plate_to_left_finger">
         <command_interface name="position">
           <param name="min">-100</param>
@@ -118,5 +118,5 @@
         </command_interface>
         <state_interface name="position"/>
-      </joint>
+      </joint> -->
     </ros2_control>
   </xacro:if>
