Commit message: Snapshot

File: description/urdf/gripper_assembly.urdf.xacro (robot description, xacro)
@@ -62,5 +62,5 @@
         <limit lower="0.15" upper="${elevator_pole_height-(elevator_connector_plate_width)}" effort="1" velocity="0.5" />
         <axis xyz="0 0 1" />
-        <dynamics damping="0.7"/>
+        <dynamics damping="0.0"/>
     </joint>
     <joint name="elevator_connector_plate_to_gripper_elevator_plate" type="fixed">

File: description/urdf/sigyn.urdf.xacro (robot description, xacro)
@@ -62,5 +62,5 @@
       name="gz::sim::systems::JointPositionController">
       <joint_name>elevator_pole_to_elevator_connector_plate</joint_name>
-      <p_gain>1.0</p_gain>
+      <p_gain>10000.0</p_gain>
       <i_gain>0.0</i_gain>
       <d_gain>0.0</d_gain>
@@ -74,5 +74,5 @@
       name="gz::sim::systems::JointPositionController">
       <joint_name>gripper_elevator_plate_to_gripper_extender</joint_name>
-      <p_gain>1.0</p_gain>
+      <p_gain>10000.0</p_gain>
       <i_gain>0.0</i_gain>
       <d_gain>0.0</d_gain>

Commit message: Snapshot

File: description/urdf/gripper_assembly.urdf.xacro (robot description, xacro)
@@ -62,5 +62,5 @@
         <limit lower="0.15" upper="${elevator_pole_height-(elevator_connector_plate_width)}" effort="1" velocity="0.5" />
         <axis xyz="0 0 1" />
-        <dynamics damping="0.0"/>
+        <dynamics damping="0.05"/>
     </joint>
     <joint name="elevator_connector_plate_to_gripper_elevator_plate" type="fixed">
@@ -108,5 +108,5 @@
         <limit lower="0" upper="${gripper_extender_length}" effort="1" velocity="0.5" />
         <axis xyz="1 0 0" />
-        <dynamics damping="0.7"/>
+        <dynamics damping="0.05"/>
     </joint>
     <xacro:colorize_link color="0.0 0.05 0.05 1.0" name="gripper_wrist_servo">
@@ -157,5 +157,5 @@
         <limit lower="-1.57" upper="1.57" effort="1" velocity="0.5" />
         <axis xyz="0 0 1" />
-        <dynamics damping="0.7"/>
+        <dynamics damping="0.02"/>
     </joint>
     <xacro:colorize_link color="${15/255} ${20/255} ${57/255} 1.0" name="left_finger">

File: description/urdf/sigyn.urdf.xacro (robot description, xacro)
@@ -62,7 +62,7 @@
       name="gz::sim::systems::JointPositionController">
       <joint_name>elevator_pole_to_elevator_connector_plate</joint_name>
-      <p_gain>10000.0</p_gain>
+      <p_gain>500.0</p_gain>
       <i_gain>0.0</i_gain>
-      <d_gain>0.0</d_gain>
+      <d_gain>50.0</d_gain>
       <i_max>0.0</i_max>
       <i_min>0.0</i_min>
@@ -74,7 +74,7 @@
       name="gz::sim::systems::JointPositionController">
       <joint_name>gripper_elevator_plate_to_gripper_extender</joint_name>
-      <p_gain>10000.0</p_gain>
+      <p_gain>500.0</p_gain>
       <i_gain>0.0</i_gain>
-      <d_gain>0.0</d_gain>
+      <d_gain>50.0</d_gain>
       <i_max>0.0</i_max>
       <i_min>0.0</i_min>

Commit message: Huzzah! First successful "fetch me a beer" run

File: description/urdf/gripper_assembly.urdf.xacro (robot description, xacro)
@@ -60,5 +60,5 @@
         <parent link="evelator_pole" />
         <child link="elevator_connector_plate" />
-        <limit lower="0.15" upper="${elevator_pole_height-(elevator_connector_plate_width)}" effort="1" velocity="0.5" />
+        <limit lower="0.15" upper="${elevator_pole_height-(elevator_connector_plate_width)}" effort="50" velocity="0.5" />
         <axis xyz="0 0 1" />
         <dynamics damping="0.05"/>
@@ -171,4 +171,20 @@
                     <box size="${finger_length} ${finger_width} ${finger_depth}" />
                 </geometry>
+                <surface>
+                    <friction>
+                        <ode>
+                            <mu>3.0</mu>
+                            <mu2>3.0</mu2>
+                            <slip1>0.01</slip1>
+                            <slip2>0.01</slip2>
+                        </ode>
+                    </friction>
+                    <contact>
+                        <ode>
+                            <kp>200000.0</kp>
+                            <kd>1.0</kd>
+                        </ode>
+                    </contact>
+                </surface>
             </collision>
             <xacro:solid_cuboid_inertial rpy="0 0 0" xyz="0 0 0" mass_kg="0.001" x="${finger_length}" y="${finger_width}" z="${finger_depth}" />
@@ -179,7 +195,7 @@
         <parent link="parallel_gripper_base_plate" />
         <child link="left_finger" />
-        <limit lower="-${(parallel_gripper_base_plate_length/2) - (finger_depth)}" upper="0" effort="1" velocity="0.5" />
-        <axis xyz="0 0 1" />
-        <dynamics damping="0.7"/>
+        <limit lower="-${(parallel_gripper_base_plate_length/2) - (finger_depth)}" upper="0" effort="200" velocity="0.5" />
+        <axis xyz="0 0 1" />
+        <dynamics damping="0.1"/>
     </joint>
     <xacro:colorize_link color="${69/255} ${16/255} ${29/255} 1.0" name="right_finger">
@@ -195,6 +211,22 @@
                     <box size="${finger_length} ${finger_width} ${finger_depth}" />
                 </geometry>
-            </collision>
-            <xacro:solid_cuboid_inertial rpy="0 0 0" xyz="0 0 0" mass_kg="0.001" x="${finger_length}" y="${finger_width}" z="${finger_depth}" />
+                <surface>
+                    <friction>
+                        <ode>
+                            <mu>3.0</mu>
+                            <mu2>3.0</mu2>
+                            <slip1>0.001</slip1>
+                            <slip2>0.001</slip2>
+                        </ode>
+                    </friction>
+                    <contact>
+                        <ode>
+                            <kp>200000.0</kp>
+                            <kd>1.0</kd>
+                        </ode>
+                    </contact>
+                </surface>
+            </collision>
+            <xacro:solid_cuboid_inertial rpy="0 0 0" xyz="0 0 0" mass_kg="0.1" x="${finger_length}" y="${finger_width}" z="${finger_depth}" />
         </foo>
     </xacro:colorize_link>
@@ -203,8 +235,7 @@
         <parent link="parallel_gripper_base_plate" />
         <child link="right_finger" />
-        <limit lower="0" upper="${(parallel_gripper_base_plate_length/2) - (finger_depth)}" effort="1" velocity="0.5" />
-        <mimic joint="parallel_gripper_base_plate_to_left_finger" multiplier="-1" offset="0" />
-        <axis xyz="0 0 1" />
-        <dynamics damping="0.7"/>
+        <limit lower="0" upper="${(parallel_gripper_base_plate_length/2) - (finger_depth)}" effort="200" velocity="0.5" />
+        <axis xyz="0 0 1" />
+        <dynamics damping="0.1"/>
     </joint>
 </robot>

File: description/urdf/ros2_control.xacro (robot description, xacro)
@@ -112,7 +112,11 @@
         <state_interface name="position"/>
       </joint>
-      <!-- <joint name="parallel_gripper_base_plate_to_right_finger">
+      <joint name="parallel_gripper_base_plate_to_right_finger">
+        <command_interface name="position">
+          <param name="min">-100</param>
+          <param name="max">100</param>
+        </command_interface>
         <state_interface name="position"/>
-      </joint> -->
+      </joint>
     </ros2_control>
   </xacro:if>

File: description/urdf/sigyn.urdf.xacro (robot description, xacro)
@@ -67,6 +67,6 @@
       <i_max>0.0</i_max>
       <i_min>0.0</i_min>
-      <cmd_max>1</cmd_max>
-      <cmd_min>-1</cmd_min>
+      <cmd_max>50</cmd_max>
+      <cmd_min>-50</cmd_min>
       <topic>/elevator_connector_plate/position</topic>
     </plugin>
@@ -98,11 +98,11 @@
       name="gz::sim::systems::JointPositionController">
       <joint_name>parallel_gripper_base_plate_to_left_finger</joint_name>
-      <p_gain>1.0</p_gain>
+      <p_gain>2000.0</p_gain>
       <i_gain>0.0</i_gain>
-      <d_gain>0.0</d_gain>
+      <d_gain>100.0</d_gain>
       <i_max>0.0</i_max>
       <i_min>0.0</i_min>
-      <cmd_max>1</cmd_max>
-      <cmd_min>-1</cmd_min>
+      <cmd_max>200</cmd_max>
+      <cmd_min>-200</cmd_min>
       <topic>/parallel_gripper_base_plate_to_left_finger/position</topic>
     </plugin>
@@ -110,11 +110,11 @@
       name="gz::sim::systems::JointPositionController">
       <joint_name>parallel_gripper_base_plate_to_right_finger</joint_name>
-      <p_gain>1.0</p_gain>
+      <p_gain>2000.0</p_gain>
       <i_gain>0.0</i_gain>
-      <d_gain>0.0</d_gain>
+      <d_gain>100.0</d_gain>
       <i_max>0.0</i_max>
       <i_min>0.0</i_min>
-      <cmd_max>1</cmd_max>
-      <cmd_min>-1</cmd_min>
+      <cmd_max>200</cmd_max>
+      <cmd_min>-200</cmd_min>
       <topic>/parallel_gripper_base_plate_to_right_finger/position</topic>
     </plugin>

Commit message: Picks up can again

File: description/urdf/gripper_assembly.urdf.xacro (robot description, xacro)
@@ -174,13 +174,12 @@
                     <friction>
                         <ode>
-                            <mu>3.0</mu>
-                            <mu2>3.0</mu2>
-                            <slip1>0.01</slip1>
-                            <slip2>0.01</slip2>
+                            <mu>100.0</mu>
+                            <mu2>100.0</mu2>
+                            <min_depth>0.001</min_depth>
                         </ode>
                     </friction>
                     <contact>
                         <ode>
-                            <kp>100000000.0</kp>
+                            <kp>10000000.0</kp>
                             <kd>1.0</kd>
                         </ode>
@@ -188,5 +187,5 @@
                 </surface>
             </collision>
-            <xacro:solid_cuboid_inertial rpy="0 0 0" xyz="0 0 0" mass_kg="0.001" x="${finger_length}" y="${finger_width}" z="${finger_depth}" />
+            <xacro:solid_cuboid_inertial rpy="0 0 0" xyz="0 0 0" mass_kg="0.1" x="${finger_length}" y="${finger_width}" z="${finger_depth}" />
         </foo>
     </xacro:colorize_link>
@@ -195,5 +194,5 @@
         <parent link="parallel_gripper_base_plate" />
         <child link="left_finger" />
-        <limit lower="-${(parallel_gripper_base_plate_length/2) - (finger_depth)}" upper="0" effort="200" velocity="0.5" />
+        <limit lower="-${(parallel_gripper_base_plate_length/2) - (finger_depth)}" upper="0" effort="1000" velocity="0.5" />
         <axis xyz="0 0 1" />
         <dynamics damping="0.1"/>
@@ -214,13 +213,12 @@
                     <friction>
                         <ode>
-                            <mu>3.0</mu>
-                            <mu2>3.0</mu2>
-                            <slip1>0.001</slip1>
-                            <slip2>0.001</slip2>
+                            <mu>100.0</mu>
+                            <mu2>100.0</mu2>
+                            <min_depth>0.001</min_depth>
                         </ode>
                     </friction>
                     <contact>
                         <ode>
-                            <kp>100000000.0</kp>
+                            <kp>10000000.0</kp>
                             <kd>1.0</kd>
                         </ode>
@@ -235,5 +233,5 @@
         <parent link="parallel_gripper_base_plate" />
         <child link="right_finger" />
-        <limit lower="0" upper="${(parallel_gripper_base_plate_length/2) - (finger_depth)}" effort="200" velocity="0.5" />
+        <limit lower="0" upper="${(parallel_gripper_base_plate_length/2) - (finger_depth)}" effort="1000" velocity="0.5" />
         <axis xyz="0 0 1" />
         <dynamics damping="0.1"/>

File: description/urdf/sigyn.urdf.xacro (robot description, xacro)
@@ -98,11 +98,11 @@
       name="gz::sim::systems::JointPositionController">
       <joint_name>parallel_gripper_base_plate_to_left_finger</joint_name>
-      <p_gain>2000.0</p_gain>
+      <p_gain>10000.0</p_gain>
       <i_gain>0.0</i_gain>
       <d_gain>100.0</d_gain>
       <i_max>0.0</i_max>
       <i_min>0.0</i_min>
-      <cmd_max>200</cmd_max>
-      <cmd_min>-200</cmd_min>
+      <cmd_max>1000</cmd_max>
+      <cmd_min>-1000</cmd_min>
       <topic>/parallel_gripper_base_plate_to_left_finger/position</topic>
     </plugin>
@@ -110,11 +110,11 @@
       name="gz::sim::systems::JointPositionController">
       <joint_name>parallel_gripper_base_plate_to_right_finger</joint_name>
-      <p_gain>2000.0</p_gain>
+      <p_gain>10000.0</p_gain>
       <i_gain>0.0</i_gain>
       <d_gain>100.0</d_gain>
       <i_max>0.0</i_max>
       <i_min>0.0</i_min>
-      <cmd_max>200</cmd_max>
-      <cmd_min>-200</cmd_min>
+      <cmd_max>1000</cmd_max>
+      <cmd_min>-1000</cmd_min>
       <topic>/parallel_gripper_base_plate_to_right_finger/position</topic>
     </plugin>

Commit message: Step3 and sim all working.

File: description/urdf/gripper_assembly.urdf.xacro (robot description, xacro)
@@ -194,7 +194,7 @@
         <parent link="parallel_gripper_base_plate" />
         <child link="left_finger" />
-        <limit lower="-${(parallel_gripper_base_plate_length/2) - (finger_depth)}" upper="0" effort="1000" velocity="0.5" />
-        <axis xyz="0 0 1" />
-        <dynamics damping="0.1"/>
+        <limit lower="-${(parallel_gripper_base_plate_length/2) - (finger_depth)}" upper="0" effort="10000" velocity="0.5" />
+        <axis xyz="0 0 1" />
+        <dynamics damping="1.0" stiffness="10000.0"/>
     </joint>
     <xacro:colorize_link color="${69/255} ${16/255} ${29/255} 1.0" name="right_finger">
@@ -233,7 +233,7 @@
         <parent link="parallel_gripper_base_plate" />
         <child link="right_finger" />
-        <limit lower="0" upper="${(parallel_gripper_base_plate_length/2) - (finger_depth)}" effort="1000" velocity="0.5" />
-        <axis xyz="0 0 1" />
-        <dynamics damping="0.1"/>
+        <limit lower="0" upper="${(parallel_gripper_base_plate_length/2) - (finger_depth)}" effort="10000" velocity="0.5" />
+        <axis xyz="0 0 1" />
+        <dynamics damping="1.0" stiffness="10000.0"/>
     </joint>
 </robot>

File: description/urdf/sim_cameras.urdf.xacro (robot description, xacro)
@@ -5,8 +5,8 @@
     <joint name="oakd_sim_joint" type="fixed">
       <parent link="${parent_link}"/>
-      <child link="oakd_sim_link"/>
+      <child link="oak-d-base-frame"/>
       <origin xyz="-0.12 -0.02 1.47" rpy="0 ${(pi / 4)+13*(2.0*pi/360.0)} ${-0*(2.0*pi/360.0)}"/>
     </joint>
-    <link name="oakd_sim_link">
+    <link name="oak-d-base-frame">
       <visual>
         <geometry>
@@ -18,11 +18,23 @@
       </visual>
     </link>
-    <joint name="oakd_sim_optical_joint" type="fixed">
-      <parent link="oakd_sim_link"/>
-      <child link="oakd_sim_optical"/>
+    <link name="oak" />
+    <joint name="oak_sim_center_joint" type="fixed">
+      <parent link="oak-d-base-frame"/>
+      <child link="oak"/>
+      <origin xyz="0 0 0" rpy="0 0 0"/>
+    </joint>
+    <link name="oak_rgb_camera_frame" />
+    <joint name="oak_rgb_camera_joint" type="fixed">
+      <parent link="oak"/>
+      <child link="oak_rgb_camera_frame"/>
+      <origin xyz="0 0 0" rpy="0 0 0"/>
+    </joint>
+    <link name="oak_rgb_camera_optical_frame" />
+    <joint name="oak_rgb_camera_optical_joint" type="fixed">
+      <parent link="oak_rgb_camera_frame"/>
+      <child link="oak_rgb_camera_optical_frame"/>
       <origin xyz="0 0 0" rpy="${-pi/2} 0 ${-pi/2}"/>
     </joint>
-    <link name="oakd_sim_optical"/>
-    <gazebo reference="oakd_sim_link">
+    <gazebo reference="oak_rgb_camera_frame">
       <sensor name="oakd_camera" type="camera">
         <pose>0 0 0 0 0 0</pose>
@@ -42,5 +54,5 @@
         </camera>
         <topic>/oakd_top/color/image</topic>
-        <gz_frame_id>oakd_sim_optical</gz_frame_id>
+        <gz_frame_id>oak_rgb_camera_optical_frame</gz_frame_id>
       </sensor>
     </gazebo>
