Commit message: Refactoring or urdfs

File: description/urdf/sigyn.urdf.xacro (robot description, xacro)
@@ -1,4 +1,5 @@
 <?xml version="1.0"?>
 <robot xmlns:xacro="http://ros.org/wiki/xacro" name="Sigyn">
+  <xacro:include filename="$(find description)/urdf/common_macros.xacro" />
   <xacro:include filename="$(find description)/urdf/inertials.xacro" />
   <xacro:property name="props" value="${xacro.load_yaml('sigyn_config.yaml')}" />

File: description/urdf/sigyn_caster_wheel_macro.urdf.xacro (robot description, xacro)
@@ -1,78 +1,4 @@
 <?xml version="1.0"?>
-<robot xmlns:xacro="http://ros.org/wiki/xacro">
-  <xacro:macro name="caster_wheel_upright" params="config name y_offset_multiplier">
-    <xacro:property name="pi" value="3.14159265359" />
-    <xacro:property name="chassis_bottom" value="${config.wheels.radius + (config.wheels.gear_box_height / 2) + config.wheels.gear_box_spacing_from_base}" />
-    <xacro:property name="upright_width" value="0.01" />
-    <xacro:property name="cf_color" value="0.7 0.7 0.72 1.0" />
-    <link name="caster_frame_${name}">
-      <visual>
-        <origin xyz="0 0 0" rpy="0 0 0" />
-        <geometry>
-          <box size="${chassis_bottom - config.caster.radius} ${upright_width} 0.005" />
-        </geometry>
-        <material name="caster_upright_color">
-          <color rgba="${cf_color}" />
-        </material>
-      </visual>
-    </link>
-    <gazebo reference="caster_frame_${name}">
-      <visual>
-        <material>
-          <ambient>${cf_color}</ambient>
-          <diffuse>${cf_color}</diffuse>
-          <specular>${cf_color}</specular>
-          <emissive>0.0 0.0 0.0 0.0</emissive>
-        </material>
-      </visual>
-    </gazebo>
-    <joint name="caster_frame_${name}_joint" type="fixed">
-      <parent link="chassis" />
-      <child link="caster_frame_${name}" />
-      <origin xyz="${-(config.body.radius - config.caster.x_offset)} ${((upright_width/2) + (config.caster.width/2)) * y_offset_multiplier} -${chassis_bottom - config.caster.radius - (chassis_bottom - config.caster.radius)/2}" rpy="${pi/2} ${pi/2} 0" />
-    </joint>
-  </xacro:macro>
-  <xacro:macro name="caster_wheel" params="config">
-    <xacro:property name="pi" value="3.14159265359" />
-    <xacro:property name="cw_color" value="0.416 0.051 0.047 1.0" />
-    <link name="caster_wheel_link">
-      <visual>
-        <origin xyz="0 0 0" rpy="0 0 0" />
-        <geometry>
-          <cylinder radius="${config.caster.radius}" length="${config.caster.width}" />
-        </geometry>
-        <material name="red">
-          <color rgba="${cw_color}" />
-        </material>
-      </visual>
-      <collision>
-        <origin xyz="0 0 0" rpy="${pi/2} 0 0" />
-        <geometry>
-          <cylinder radius="${config.caster.radius}" length="${config.caster.width}" />
-        </geometry>
-      </collision>
-      <xacro:solid_cylinder_inertial rpy="0 0 0" xyz="0 0 0" mass_kg="${config.caster.mass}" radius="${config.caster.radius}" length="${config.caster.width}" />
-    </link>
-    <gazebo reference="caster_wheel_link">
-      <mu1>0.01</mu1>
-      <mu2>0.01</mu2>
-      <visual>
-        <material>
-          <ambient>${cw_color}</ambient>
-          <diffuse>${cw_color}</diffuse>
-          <specular>${cw_color}</specular>
-          <emissive>0.0 0.0 0.0 0.0</emissive>
-        </material>
-      </visual>
-    </gazebo>
-    <joint name="caster_wheel_joint" type="fixed">
-      <parent link="chassis" />
-      <child link="caster_wheel_link" />
-      <origin xyz="${-(config.body.radius - config.caster.x_offset)} 0 -${config.wheels.radius + (config.wheels.gear_box_height / 2) -config.caster.radius + config.wheels.gear_box_spacing_from_base}" rpy="${pi/2} 0 0" />
-    </joint>
-    <xacro:caster_wheel_upright config="${config}" name="left" y_offset_multiplier="1" />
-    <xacro:caster_wheel_upright config="${config}" name="right" y_offset_multiplier="-1" />
-  </xacro:macro>
-  <!--
+<!--
 Copyright (c) 2024 Michael Wimble
 Permission is hereby granted, free of charge, to any person obtaining a copy
@@ -92,3 +18,51 @@
 SOFTWARE.
 -->
+<robot xmlns:xacro="http://ros.org/wiki/xacro">
+  <xacro:macro name="caster_wheel_upright" params="config name y_offset_multiplier">
+    <xacro:property name="chassis_bottom" value="${config.wheels.radius + (config.wheels.gear_box_height / 2) + config.wheels.gear_box_spacing_from_base}" />
+    <xacro:property name="upright_width" value="0.01" />
+    <xacro:colorize_link color="0.7 0.7 0.72 1.0" name="caster_frame_${name}">
+      <foo>
+        <visual>
+          <origin xyz="0 0 0" rpy="0 0 0" />
+          <geometry>
+            <box size="${chassis_bottom - config.caster.radius} ${upright_width} 0.005" />
+          </geometry>
+          <material name="caster_frame_${name}"/>
+        </visual>
+      </foo>
+    </xacro:colorize_link>
+    <joint name="caster_frame_${name}_joint" type="fixed">
+      <parent link="chassis" />
+      <child link="caster_frame_${name}" />
+      <origin xyz="${-(config.body.radius - config.caster.x_offset)} ${((upright_width/2) + (config.caster.width/2)) * y_offset_multiplier} -${chassis_bottom - config.caster.radius - (chassis_bottom - config.caster.radius)/2}" rpy="${pi/2} ${pi/2} 0" />
+    </joint>
+  </xacro:macro>
+  <xacro:macro name="caster_wheel" params="config">
+    <xacro:colorize_link color="0.416 0.051 0.047 1.0" name="caster_wheel_link">
+      <foo>
+        <visual>
+          <origin xyz="0 0 0" rpy="0 0 0" />
+          <geometry>
+            <cylinder radius="${config.caster.radius}" length="${config.caster.width}" />
+          </geometry>
+          <material name="caster_wheel_link"/>
+        </visual>
+        <collision>
+          <origin xyz="0 0 0" rpy="${pi/2} 0 0" />
+          <geometry>
+            <cylinder radius="${config.caster.radius}" length="${config.caster.width}" />
+          </geometry>
+        </collision>
+        <xacro:solid_cylinder_inertial rpy="0 0 0" xyz="0 0 0" mass_kg="${config.caster.mass}" radius="${config.caster.radius}" length="${config.caster.width}" />
+      </foo>
+    </xacro:colorize_link>
+    <joint name="caster_wheel_joint" type="fixed">
+      <parent link="chassis" />
+      <child link="caster_wheel_link" />
+      <origin xyz="${-(config.body.radius - config.caster.x_offset)} 0 -${config.wheels.radius + (config.wheels.gear_box_height / 2) -config.caster.radius + config.wheels.gear_box_spacing_from_base}" rpy="${pi/2} 0 0" />
+    </joint>
+    <xacro:caster_wheel_upright config="${config}" name="left" y_offset_multiplier="1" />
+    <xacro:caster_wheel_upright config="${config}" name="right" y_offset_multiplier="-1" />
+  </xacro:macro>
 </robot>

File: description/urdf/sigyn_wheels_macro.urdf.xacro (robot description, xacro)
@@ -1,108 +1,4 @@
 <?xml version="1.0"?>
-<robot xmlns:xacro="http://ros.org/wiki/xacro">
-  <xacro:macro name="wheel" params="axis side radius width pos_x pos_y pos_z mass_kg">
-    <!-- Create the outer, rubber tire -->
-    <link name="${side}_wheel_link">
-      <visual name="tire">
-        <origin xyz="0 0 0" rpy="0 0 0" />
-        <geometry>
-          <cylinder radius="${radius}" length="${width - 0.004}" />
-        </geometry>
-        <material name="wheel_black">
-          <color rgba="0.15 0.15 0.15 1.0" />
-        </material>
-      </visual>
-      <collision>
-        <origin xyz="0 0 0" rpy="${pi/2} 0 0" />
-        <geometry>
-          <cylinder radius="${radius}" length="${width}" />
-        </geometry>
-      </collision>
-      <xacro:solid_cylinder_inertial rpy="${pi/2} 0 0" xyz="0 0 0" mass_kg="${mass_kg}" radius="${radius}" length="${width}" />
-    </link>
-    <gazebo reference="${side}_wheel_link">
-      <visual>
-        <material>
-          <ambient>0.15 0.15 0.15 1.0</ambient>
-          <diffuse>0.15 0.15 0.15 1.0</diffuse>
-          <specular>0.15 0.15 0.15 1.0</specular>
-          <emissive>0.0 0.0 0.0 0.0</emissive>
-        </material>
-      </visual>
-    </gazebo>
-    <joint name="${side}_wheel_joint" type="continuous">
-      <axis xyz="0 0 ${axis}" />
-      <parent link="base_link" />
-      <child link="${side}_wheel_link" />
-      <origin xyz="${pos_x} ${pos_y} ${pos_z}" rpy="${-axis * pi / 2} 0 0" />
-    </joint>
-    <!-- Create the wheel hub -->
-    <link name="${side}_wheel_hub">
-      <origin xyz="0 0 0" rpy="0 0 0" />
-      <visual>
-        <geometry>
-          <cylinder radius="${radius - 0.02}" length="${width - 0.002}" />
-        </geometry>
-        <material name="wheel_silver">
-          <color rgba="0.8 0.8 0.8 1.0" />
-        </material>
-      </visual>
-    </link>
-    <gazebo reference="${side}_wheel_hub">
-      <visual>
-        <material>
-          <ambient>0.8 0.8 0.8 1.0</ambient>
-          <diffuse>0.8 0.8 0.8 1.0</diffuse>
-          <specular>0.8 0.8 0.8 1.0</specular>
-          <emissive>0.0 0.0 0.0 0.0</emissive>
-        </material>
-      </visual>
-    </gazebo>
-    <joint name="${side}_wheel_hub_joint" type="fixed">
-      <axis xyz="0 0 ${axis}" />
-      <parent link="${side}_wheel_link" />
-      <child link="${side}_wheel_hub" />
-      <origin xyz="0 0 0" rpy="0 0 0" />
-    </joint>
-    <!-- Create the wheel marker -->
-    <link name="${side}_wheel_marker">
-      <origin xyz="0 0 0" rpy="0 0 0" />
-      <visual>
-        <geometry>
-          <box size="0.01 ${(radius / 2)} ${width}" />
-        </geometry>
-        <material name="wheel_marker">
-          <color rgba="0.86 0.54 0.86 1" />
-        </material>
-      </visual>
-    </link>
-    <gazebo reference="${side}_wheel_marker">
-      <visual>
-        <material>
-          <ambient>0.86 0.54 0.86 1.0</ambient>
-          <diffuse>0.86 0.54 0.86 1.0</diffuse>
-          <specular>0.86 0.54 0.86 1.0</specular>
-          <emissive>0.0 0.0 0.0 0.0</emissive>
-        </material>
-      </visual>
-    </gazebo>
-    <joint name="${side}_wheel_marker_joint" type="fixed">
-      <parent link="${side}_wheel_hub" />
-      <child link="${side}_wheel_marker" />
-      <origin xyz="0 ${(radius - 0.02) / 2} 0" rpy="0 0 0" />
-    </joint>
-  </xacro:macro>
-  <xacro:macro name="wheels" params="config instances:=^*">
-    <xacro:if value="${instances}">
-      <!-- pop first item from list -->
-      <xacro:property name="instance" value="${instances.pop(0)}"/>
-      <foo instance="${instance['name']}"/>
-      <xacro:property name="y" value="${(config.body.radius-config.wheels.center_offset)*instance['y_position_multiplier']}"/>
-      <xacro:property name="z" value="-${(config.wheels.gear_box_height/2)+config.wheels.gear_box_spacing_from_base}"/>
-      <xacro:wheel axis="${instance['y_position_multiplier']}" pos_y="${y}" pos_z="${z}" side="${instance['name']}" radius="${config.wheels.radius}" width="${config.wheels.width}" pos_x="0.0" mass_kg="${config.wheels.mass}" />
-      <xacro:wheels config="${config}" instances="${instances}"/>
-    </xacro:if>
-  </xacro:macro>
-  <!--
+<!--
 Copyright (c) 2024 Michael Wimble
 Permission is hereby granted, free of charge, to any person obtaining a copy
@@ -122,3 +18,76 @@
 SOFTWARE.
 -->
+<robot xmlns:xacro="http://ros.org/wiki/xacro">
+  <xacro:macro name="wheel" params="axis side radius width pos_x pos_y pos_z mass_kg">
+    <!-- Create the outer, rubber tire -->
+    <xacro:colorize_link color="0.15 0.15 0.15 1.0" name="${side}_wheel_link">
+      <foo>
+        <visual name="tire">
+          <origin xyz="0 0 0" rpy="0 0 0" />
+          <geometry>
+            <cylinder radius="${radius}" length="${width - 0.004}" />
+          </geometry>
+          <material name="${side}_wheel_link"/>
+        </visual>
+        <collision>
+          <origin xyz="0 0 0" rpy="${pi/2} 0 0" />
+          <geometry>
+            <cylinder radius="${radius}" length="${width}" />
+          </geometry>
+        </collision>
+        <xacro:solid_cylinder_inertial rpy="${pi/2} 0 0" xyz="0 0 0" mass_kg="${mass_kg}" radius="${radius}" length="${width}" />
+      </foo>
+    </xacro:colorize_link>
+    <joint name="${side}_wheel_joint" type="continuous">
+      <axis xyz="0 0 ${axis}" />
+      <parent link="base_link" />
+      <child link="${side}_wheel_link" />
+      <origin xyz="${pos_x} ${pos_y} ${pos_z}" rpy="${-axis * pi / 2} 0 0" />
+    </joint>
+    <!-- Create the wheel hub -->
+    <xacro:colorize_link color="0.8 0.8 0.8 1.0" name="${side}_wheel_hub">
+      <foo>
+        <origin xyz="0 0 0" rpy="0 0 0" />
+        <visual>
+          <geometry>
+            <cylinder radius="${radius - 0.02}" length="${width - 0.002}" />
+          </geometry>
+          <material name="${side}_wheel_hub"/>
+        </visual>
+      </foo>
+    </xacro:colorize_link>
+    <joint name="${side}_wheel_hub_joint" type="fixed">
+      <axis xyz="0 0 ${axis}" />
+      <parent link="${side}_wheel_link" />
+      <child link="${side}_wheel_hub" />
+      <origin xyz="0 0 0" rpy="0 0 0" />
+    </joint>
+    <!-- Create the wheel marker -->
+    <xacro:colorize_link color="0.86 0.54 0.86 1" name="${side}_wheel_marker">
+      <foo>
+        <origin xyz="0 0 0" rpy="0 0 0" />
+        <visual>
+          <geometry>
+            <box size="0.01 ${(radius / 2)} ${width}" />
+          </geometry>
+          <material name="${side}_wheel_marker"/>
+        </visual>
+      </foo>
+    </xacro:colorize_link>
+    <joint name="${side}_wheel_marker_joint" type="fixed">
+      <parent link="${side}_wheel_hub" />
+      <child link="${side}_wheel_marker" />
+      <origin xyz="0 ${(radius - 0.02) / 2} 0" rpy="0 0 0" />
+    </joint>
+  </xacro:macro>
+  <xacro:macro name="wheels" params="config instances:=^*">
+    <xacro:if value="${instances}">
+      <!-- pop first item from list -->
+      <xacro:property name="instance" value="${instances.pop(0)}"/>
+      <xacro:property name="y" value="${(config.body.radius-config.wheels.center_offset)*instance['y_position_multiplier']}"/>
+      <xacro:property name="z" value="-${(config.wheels.gear_box_height/2)+config.wheels.gear_box_spacing_from_base}"/>
+      <xacro:wheel axis="${instance['y_position_multiplier']}" pos_y="${y}" pos_z="${z}" side="${instance['name']}" radius="${config.wheels.radius}" width="${config.wheels.width}" pos_x="0.0" mass_kg="${config.wheels.mass}" />
+      <xacro:wheels config="${config}" instances="${instances}"/>
+    </xacro:if>
+  </xacro:macro>
 </robot>

Commit message: Temp addition of lidar and diff_drive_controller

File: description/urdf/sigyn.urdf.xacro (robot description, xacro)
@@ -13,3 +13,8 @@
   <!-- Make the caster wheel -->
   <xacro:caster_wheel config="${props}" />
+  <xacro:include filename="$(find description)/urdf/properties.urdf.xacro" />
+  <xacro:ld06 lidar_prefix="top_lidar">
+    <origin xyz="0.155 0 0.300" rpy="0 0 -${pi / 2}" />
+  </xacro:ld06>
+  <xacro:diff_drive_controller wheel_separation="${wheel_pos_y * 2}" wheel_radius="${wheel_radius}" />
 </robot>

Commit message: Misc tweaks

File: description/urdf/sigyn.urdf.xacro (robot description, xacro)
@@ -38,5 +38,5 @@
   <!-- <xacro:oakd_link mount_point="elevator_top" /> -->
   <xacro:oakd_joint mount_point="elevator_top">
-    <origin xyz="-0.12 -0.02 1.5" rpy="0 ${(pi / 4)+9*(2.0*pi/360.0)} ${-9*(2.0*pi/360.0)}" />
+    <origin xyz="-0.12 -0.02 1.45" rpy="0 ${(pi / 4)+9*(2.0*pi/360.0)} ${-9*(2.0*pi/360.0)}" />
   </xacro:oakd_joint>
   <gazebo>

Commit message: Fixes for stereo local map addition.

File: description/urdf/sigyn.urdf.xacro (robot description, xacro)
@@ -38,5 +38,5 @@
   <!-- <xacro:oakd_link mount_point="elevator_top" /> -->
   <xacro:oakd_joint mount_point="elevator_top">
-    <origin xyz="-0.12 -0.02 1.45" rpy="0 ${(pi / 4)+9*(2.0*pi/360.0)} ${-9*(2.0*pi/360.0)}" />
+    <origin xyz="-0.12 -0.02 1.6" rpy="0 ${(pi / 4)+9*(2.0*pi/360.0)} ${-9*(2.0*pi/360.0)}" /> <!--was 1.45 -->
   </xacro:oakd_joint>
   <gazebo>

Commit message: Finder positioning of OAK-D

File: description/urdf/sigyn.urdf.xacro (robot description, xacro)
@@ -38,5 +38,5 @@
   <!-- <xacro:oakd_link mount_point="elevator_top" /> -->
   <xacro:oakd_joint mount_point="elevator_top">
-    <origin xyz="-0.12 -0.02 1.6" rpy="0 ${(pi / 4)+9*(2.0*pi/360.0)} ${-9*(2.0*pi/360.0)}" /> <!--was 1.45 -->
+    <origin xyz="-0.12 -0.02 1.47" rpy="0 ${(pi / 4)+13*(2.0*pi/360.0)} ${-0*(2.0*pi/360.0)}" /> <!--was 1.45 -->
   </xacro:oakd_joint>
   <gazebo>

Commit message: Restore pi_servo1 package from commit 6fa3b46

File: description/urdf/sigyn.urdf.xacro (robot description, xacro)
@@ -38,5 +38,5 @@
   <!-- <xacro:oakd_link mount_point="elevator_top" /> -->
   <xacro:oakd_joint mount_point="elevator_top">
-    <origin xyz="-0.12 -0.02 1.47" rpy="0 ${(pi / 4)+13*(2.0*pi/360.0)} ${-0*(2.0*pi/360.0)}" /> <!--was 1.45 -->
+    <origin xyz="-0.12 -0.02 1.47" rpy="0 ${(pi / 4)+13*(2.0*pi/360.0)} ${-0*(2.0*pi/360.0)}" />
   </xacro:oakd_joint>
   <gazebo>
@@ -104,3 +104,17 @@
   <xacro:diff_drive_controller config="${props}" instances1="${props.wheels.instances}"
     instances2="${props.wheels.instances}" />
+  <!-- IMU0 - Upside down (components facing down) -->
+  <joint name="imu0_joint" type="fixed">
+    <parent link="base_link" />
+    <child link="imu0_link" />
+    <origin xyz="-0.100 0.180 0.022" rpy="0 3.14159 0" />  <!-- 180° around Y-axis -->
+  </joint>
+  <link name="imu0_link" />
+  <!-- IMU1 - Right-side up (components facing up) -->
+  <joint name="imu1_joint" type="fixed">
+    <parent link="base_link" />
+    <child link="imu1_link" />
+    <origin xyz="0.085 -0.185 0.022" rpy="0 0 0" />  <!-- No rotation needed -->
+  </joint>
+  <link name="imu1_link" />
 </robot>

Commit message: Topic analysis, beginning of ekf fix for IMUs

File: description/urdf/sigyn.urdf.xacro (robot description, xacro)
@@ -107,14 +107,14 @@
   <joint name="imu0_joint" type="fixed">
     <parent link="base_link" />
-    <child link="imu0_link" />
+    <child link="imu_0" />
     <origin xyz="-0.100 0.180 0.022" rpy="0 3.14159 0" />  <!-- 180° around Y-axis -->
   </joint>
-  <link name="imu0_link" />
+  <link name="imu_0" />
   <!-- IMU1 - Right-side up (components facing up) -->
   <joint name="imu1_joint" type="fixed">
     <parent link="base_link" />
-    <child link="imu1_link" />
+    <child link="imu_1" />
     <origin xyz="0.085 -0.185 0.022" rpy="0 0 0" />  <!-- No rotation needed -->
   </joint>
-  <link name="imu1_link" />
+  <link name="imu_1" />
 </robot>

Commit message: Faster recovery. Better MPPI tuning.

File: description/urdf/sigyn.urdf.xacro (robot description, xacro)
@@ -1,7 +1,4 @@
 <?xml version="1.0"?>
 <robot xmlns:xacro="http://ros.org/wiki/xacro" name="Sigyn">
-  <self_collide>false</self_collide>
-  <pose>0 0 0.2 0 0 0</pose>
-  <static>false</static>
   <xacro:arg name="use_ros2_control" default="true" />
   <xacro:arg name="sim_mode" default="false" />
@@ -41,6 +38,5 @@
   </xacro:oakd_joint>
   <gazebo>
-    <plugin filename="gz-sim-joint-position-controller-system"
-      name="gz::sim::systems::JointPositionController">
+    <plugin filename="gz-sim-joint-position-controller-system" name="gz::sim::systems::JointPositionController">
       <joint_name>elevator_pole_to_elevator_connector_plate</joint_name>
       <p_gain>1.0</p_gain>
@@ -53,6 +49,5 @@
       <topic>/elevator_connector_plate/position</topic>
     </plugin>
-    <plugin filename="gz-sim-joint-position-controller-system"
-      name="gz::sim::systems::JointPositionController">
+    <plugin filename="gz-sim-joint-position-controller-system" name="gz::sim::systems::JointPositionController">
       <joint_name>gripper_elevator_plate_to_gripper_extender</joint_name>
       <p_gain>1.0</p_gain>
@@ -65,6 +60,5 @@
       <topic>/gripper_elevator_plate_to_gripper_extender/position</topic>
     </plugin>
-    <plugin filename="gz-sim-joint-position-controller-system"
-      name="gz::sim::systems::JointPositionController">
+    <plugin filename="gz-sim-joint-position-controller-system" name="gz::sim::systems::JointPositionController">
       <joint_name>gripper_wrist_to_parallel_gripper_base_plate</joint_name>
       <p_gain>1.0</p_gain>
@@ -77,6 +71,5 @@
       <topic>/gripper_wrist_to_parallel_gripper_base_plate/position</topic>
     </plugin>
-    <plugin filename="gz-sim-joint-position-controller-system"
-      name="gz::sim::systems::JointPositionController">
+    <plugin filename="gz-sim-joint-position-controller-system" name="gz::sim::systems::JointPositionController">
       <joint_name>parallel_gripper_base_plate_to_left_finger</joint_name>
       <p_gain>1.0</p_gain>
@@ -89,6 +82,5 @@
       <topic>/parallel_gripper_base_plate_to_left_finger/position</topic>
     </plugin>
-    <plugin filename="gz-sim-joint-position-controller-system"
-      name="gz::sim::systems::JointPositionController">
+    <plugin filename="gz-sim-joint-position-controller-system" name="gz::sim::systems::JointPositionController">
       <joint_name>parallel_gripper_base_plate_to_right_finger</joint_name>
       <p_gain>1.0</p_gain>
@@ -102,11 +94,11 @@
     </plugin>
   </gazebo>
-  <xacro:diff_drive_controller config="${props}" instances1="${props.wheels.instances}"
-    instances2="${props.wheels.instances}" />
+  <xacro:diff_drive_controller config="${props}" instances1="${props.wheels.instances}" instances2="${props.wheels.instances}" />
   <!-- IMU0 - Upside down (components facing down) -->
   <joint name="imu0_joint" type="fixed">
     <parent link="base_link" />
     <child link="imu_0" />
-    <origin xyz="-0.100 0.180 0.022" rpy="0 3.14159 0" />  <!-- 180° around Y-axis -->
+    <origin xyz="-0.100 0.180 0.022" rpy="0 3.14159 0" />
+    <!-- 180° around Y-axis -->
   </joint>
   <link name="imu_0" />
@@ -115,5 +107,6 @@
     <parent link="base_link" />
     <child link="imu_1" />
-    <origin xyz="0.085 -0.185 0.022" rpy="0 0 0" />  <!-- No rotation needed -->
+    <origin xyz="0.085 -0.185 0.022" rpy="0 0 0" />
+    <!-- No rotation needed -->
   </joint>
   <link name="imu_1" />

Commit message: Snapshot. Lidar localization working again.

File: description/urdf/sigyn.urdf.xacro (robot description, xacro)
@@ -98,18 +98,16 @@
   </gazebo>
   <xacro:diff_drive_controller config="${props}" instances1="${props.wheels.instances}" instances2="${props.wheels.instances}" />
-  <!-- IMU0 - Upside down (components facing down) -->
+  <!-- IMU0 - Upside down & backwards -->
   <joint name="imu0_joint" type="fixed">
     <parent link="base_link" />
     <child link="imu_0" />
-    <origin xyz="-0.100 0.180 0.022" rpy="0 3.14159 0" />
-    <!-- 180° around Y-axis -->
+    <origin xyz="-0.100 0.180 0.022" rpy="0 3.14159 3.14159" />
   </joint>
   <link name="imu_0" />
-  <!-- IMU1 - Right-side up (components facing up) -->
+  <!-- IMU1 - Right-side up & backwards -->
   <joint name="imu1_joint" type="fixed">
     <parent link="base_link" />
     <child link="imu_1" />
-    <origin xyz="0.085 -0.185 0.022" rpy="0 0 0" />
-    <!-- No rotation needed -->
+    <origin xyz="0.085 -0.185 0.022" rpy="0 0 3.14159" />
   </joint>
   <link name="imu_1" />
