Commit message: Fixes for do_top_lidar:=false

File: description/urdf/sigyn.urdf.xacro (robot description, xacro)
@@ -3,4 +3,5 @@
   <xacro:arg name="use_ros2_control" default="true" />
   <xacro:arg name="sim_mode" default="false" />
+  <xacro:arg name="do_top_lidar" default="true" />
   <xacro:include filename="$(find description)/urdf/common_macros.xacro" />
   <xacro:include filename="$(find description)/urdf/inertials.xacro" />
@@ -28,10 +29,20 @@
   <xacro:caster_wheel config="${props}" />
   <xacro:include filename="$(find description)/urdf/ld06.urdf.xacro" />
-  <xacro:ld06 lidar_prefix="top_lidar" topic_name="scan">
-    <origin xyz="0.155 0 0.300" rpy="0 0 -${pi / 2}" />
-  </xacro:ld06>
-  <xacro:ld06 lidar_prefix="cup_lidar" topic_name="scan_cup">
-    <origin xyz="${0.155-0.34} 0 ${0.300+1.485}" rpy="0 0 0" />
-  </xacro:ld06>
+  <!-- LiDAR configuration: if do_top_lidar=true, use both top_lidar and cup_lidar as-is.
+       if do_top_lidar=false, create only a top_lidar at the cup_lidar origin so downstream
+       code continues to use the 'top_lidar' name and 'scan' topic. -->
+  <xacro:if value="$(arg do_top_lidar)">
+    <xacro:ld06 lidar_prefix="top_lidar" topic_name="scan">
+      <origin xyz="${0.155-0.34} 0 ${0.300+1.485}" rpy="0 0 0" />
+    </xacro:ld06>
+    <xacro:ld06 lidar_prefix="cup_lidar" topic_name="scan_cup">
+      <origin xyz="0.155 0 0.300" rpy="0 0 -${pi / 2}" />
+    </xacro:ld06>
+  </xacro:if>
+  <xacro:unless value="$(arg do_top_lidar)">
+    <xacro:ld06 lidar_prefix="top_lidar" topic_name="scan">
+      <origin xyz="0.155 0 0.300" rpy="0 0 -${pi / 2}" />
+    </xacro:ld06>
+  </xacro:unless>
   <xacro:include filename="$(find description)/urdf/gazebo.urdf.xacro" />
   <xacro:include filename="$(find description)/urdf/gripper_assembly.urdf.xacro" />

Commit message: Sorta works but can sometimes take to long to provide ranged point of the object.

File: description/urdf/sigyn.urdf.xacro (robot description, xacro)
@@ -55,5 +55,5 @@
   <xacro:unless value="$(arg sim_mode)">
     <xacro:oakd_joint mount_point="elevator_top">
-      <origin xyz="-0.12 -0.02 1.47" rpy="0 ${(pi / 4)+13*(2.0*pi/360.0)} ${-0*(2.0*pi/360.0)}" />
+      <origin xyz="-0.0625 0.0 1.47" rpy="0 ${(pi / 4)+13*(2.0*pi/360.0)} ${-0*(2.0*pi/360.0)}" />
     </xacro:oakd_joint>
   </xacro:unless>

Commit message: Working snapshot

File: description/urdf/sigyn.urdf.xacro (robot description, xacro)
@@ -55,5 +55,5 @@
   <xacro:unless value="$(arg sim_mode)">
     <xacro:oakd_joint mount_point="elevator_top">
-      <origin xyz="-0.0625 0.0 1.47" rpy="0 ${(pi / 4)+13*(2.0*pi/360.0)} ${-0*(2.0*pi/360.0)}" />
+      <origin xyz="-0.0625 0.0 1.47" rpy="${-(90*pi/180.0)} ${-27.5*pi/180.0} 0" />
     </xacro:oakd_joint>
   </xacro:unless>

Commit message: Snapshot. Almost works except arm extension is backwards.

File: description/urdf/sigyn.urdf.xacro (robot description, xacro)
@@ -34,5 +34,5 @@
   <xacro:if value="$(arg do_top_lidar)">
     <xacro:ld06 lidar_prefix="top_lidar" topic_name="scan">
-      <origin xyz="${0.155-0.34} 0 ${0.300+1.485}" rpy="0 0 0" />
+      <origin xyz="${0.155-0.34} 0 ${1.485}" rpy="0 0 0" />
     </xacro:ld06>
     <xacro:ld06 lidar_prefix="cup_lidar" topic_name="scan_cup">
@@ -55,5 +55,5 @@
   <xacro:unless value="$(arg sim_mode)">
     <xacro:oakd_joint mount_point="elevator_top">
-      <origin xyz="-0.0625 0.0 1.47" rpy="${-(90*pi/180.0)} ${-27.5*pi/180.0} 0" />
+      <origin xyz="-0.0625 0.0 1.665" rpy="${-(90*pi/180.0)} ${-27.5*pi/180.0} 0" />
     </xacro:oakd_joint>
   </xacro:unless>
