Commit message: sigyn.launch.py: new starting coordinates. home.world, wall.xacro, model.sdf.xacro: for harmonic gazebo

File: description/models/home/model.sdf.xacro (robot description, xacro)
@@ -1,4 +1,4 @@
 <robot xmlns:xacro="http://ros.org/wiki/xacro" name="foo3">
-  <xacro:include filename="marker.xacro" />
+  <!-- <xacro:include filename="marker.xacro" /> -->
   <xacro:include filename="wall.xacro" />
   <sdf version="1.4">
@@ -6,5 +6,5 @@
       <static>true</static>
       <xacro:property name="wall_width" value="4" />
-      <xacro:marker name="x_origin_marker" x="0.2" y="0.3" />
+      <!-- <xacro:marker name="x_origin_marker" x="0.2" y="0.3" /> -->
       <!-- big outer walls-->
       <xacro:property name="house_ew_length" value="${(50*12)+7}" />

File: description/models/home/wall.xacro (robot description, xacro)
@@ -11,5 +11,18 @@
     <link name="${name}">
       <pose> ${x_pos_m } ${y_pos_m } ${z_pos_m} 0 0 ${rot_deg}</pose>
-      <collision name="collision">
+      <visual name='visual'>
+        <geometry>
+          <box>
+            <size>${l_m} ${w_m} ${h_m}</size>
+          </box>
+        </geometry>
+        <!--let's add color to our link-->
+        <material>
+          <ambient>1.0 0.7451 0.4353 1</ambient>
+          <diffuse>1.0 0.7451 0.4353 1</diffuse>
+          <specular>1 1 1 1</specular>
+        </material>
+      </visual>
+      <collision name='collision'>
         <geometry>
           <box>
@@ -18,17 +31,4 @@
         </geometry>
       </collision>
-      <visual name="visual">
-        <cast_shadows>false</cast_shadows>
-        <geometry>
-          <box>
-            <size>${l_m} ${w_m} ${h_m}</size>
-          </box>
-        </geometry>
-        <material>
-          <ambient>1.0 0.7451 0.4353 1</ambient>
-          <diffuse>1.0 0.7451 0.4353 1</diffuse>
-          <specular>1 1 1 1</specular>
-        </material>
-      </visual>
     </link>
   </xacro:macro>
